File: _autosave-Alpha_Breakout.kicad_pcb (KiCad board)
At the start: 2 copper layers, 4 parts, among them SW1 SW_Push, SW2 SW_Push, U1 CH340N, U2 STM32F103C8Tx

Commit message: adcs
Parts:
- added U3: ADS7828, Package_SO:TSSOP-16_4.4x5mm_P0.65mm, F.Cu at (154.3, 119.8)
- added U4: ADS7828, Package_SO:TSSOP-16_4.4x5mm_P0.65mm, F.Cu at (154.3, 126.4)
