File: _autosave-Alpha_Breakout.kicad_pcb (KiCad board)
At the start: 2 copper layers, 27 parts, among them J2 Conn_01x02, SW1 SW_Push, SW2 SW_Push, U1 CH340N, U2 STM32F103C8Tx, U3 ADS7828, U4 ADS7828, U5 AP63203WU

Commit message: reg🟡
Parts:
- added C12: .1uF, Capacitor_SMD:C_0402_1005Metric, F.Cu at (176.5, 120.4)
- added J2: Conn_01x02, TerminalBlock_Phoenix:TerminalBlock_Phoenix_MKDS-1,5-2-5.08_1x02_P5.08mm_Horizontal, F.Cu at (169.9, 113.6)
- added U5: MAX31856, Package_SO:TSSOP-14_4.4x5mm_P0.65mm, F.Cu at (170.7, 122.8)
- renumbered C16 to C15, C17 to C16, C27 to C17, C28 to C21, C21 to C22, C29 to C23, C22 to C24, C23 to C25, C30 to C26, C24 to C27, C25 to C28, C26 to C29, J2 to J3, L3 to L1, L4 to L2, R15 to R10, R13 to R8, SW2 to SW1, SW1 to SW2, U2 to U1, U1 to U2, U5 to U6
Connections:
- U1 pad 15: unconnected-(U2-PA5-Pad15) -> /stm32f1/SPI1_SCK
- U1 pad 16: unconnected-(U2-PA6-Pad16) -> /stm32f1/SPI1_MISO
- U1 pad 17: unconnected-(U2-PA7-Pad17) -> /stm32f1/SPI1_MOSI
