File: _autosave-Alpha_Breakout.kicad_pcb (KiCad board)
At the start: 2 copper layers, 66.7 x 73.7 mm, 127 parts, among them IC1 LM66200DRLR, J1 USB_C_Receptacle_USB2.0_14P, J10 Conn_01x03, J11 Conn_01x03, J12 Conn_01x03, J13 Conn_01x03, J14 Conn_01x03, J15 Conn_01x03, J16 Conn_01x03, J18 Conn_01x03, J2 Conn_01x02, J20 Conn_01x02, J21 Conn_01x02, J22 Conn_01x02, J23 Conn_01x02, J24 Conn_01x04, J25 Conn_01x02, J26 Conn_01x02, J27 Conn_01x02, J28 Conn_01x02, J29 Conn_01x02, J3 Conn_01x02, J31 Conn_01x02, J32 Conn_01x02, J33 Conn_01x02, J6 Conn_01x03, J7 Conn_01x03, J8 Conn_01x03, J9 Conn_01x03, Q1 CSD13381F4, Q2 CSD13381F4, Q3 CSD13381F4, Q4 CSD13381F4, SW1 SW_Push, SW2 SW_Push, U1 STM32F103C8Tx, U10 MAX31856, U11 SP3485EN, U12 L78L10_SOT89, U13 ADS1231ID, U2 CH340N, U3 ADS7828, U4 ADS7828, U5 MAX31856, U6 AP63203WU, U7 LP2985-3.3, U8 MAX31856, U9 MAX31856

Commit message: added leds🔴🟡🔵
Parts:
- renumbered C33 to C1, C39 to C10, C34 to C11, C1 to C12, C35 to C13, C41 to C14, C36 to C15, C42 to C16, C37 to C17, C43 to C18, C38 to C19, C40 to C20, C10 to C21, C44 to C22, C11 to C23, C45 to C24, C12 to C25, C46 to C26, C13 to C27, C47 to C28, C14 to C29, C15 to C30, C16 to C31, C17 to C32, C18 to C33, C19 to C34, C20 to C35, C21 to C36, C22 to C37, C23 to C38, C24 to C39, C25 to C40, C26 to C41, C27 to C42, C28 to C43, C29 to C44, C30 to C45, C31 to C46, C32 to C47, D5 to D1, D7 to D2, D6 to D3, D8 to D4, D1 to D5, D2 to D6, D3 to D7, D4 to D8, J8 to J10, J9 to J11, J16 to J12, J10 to J14, J11 to J15, J18 to J16, J21 to J18, J20 to J19, J22 to J20, J2 to J21, J3 to J22, J33 to J25, J25 to J26, J26 to J27, J27 to J28, J28 to J29, J6 to J3, J29 to J31, J31 to J32, J32 to J33, J12 to J4, J13 to J5, J14 to J8, J15 to J9, R16 to R10, R17 to R11, R6 to R12, R7 to R13, R8 to R14, R10 to R16, R20 to R19, R19 to R20, R14 to R6, R15 to R7, R12 to R8, R13 to R9, U7 to U10, U13 to U12, U9 to U5, U8 to U6, U10 to U7, U5 to U8, U6 to U9
Connections:
- U12 pad 1: unconnected-(U13-DVDD-Pad1) -> +3.3V
- U12 pad 10: unconnected-(U13-VREFP-Pad10) -> +5V
- U12 pad 11: Net-(U13-GND-Pad11) -> GND
- U12 pad 13: unconnected-(U13-AVDD-Pad13) -> +5V
- U12 pad 14: unconnected-(U13-~{PDWN}-Pad14) -> Net-(U12-SPEED)
- U12 pad 15: unconnected-(U13-SCLK-Pad15) -> /ADS1231/LC_SCLK
- U12 pad 16: unconnected-(U13-~{DRDY}/DOUT-Pad16) -> /ADS1231/LC_DRDY/DOUT
- U12 pad 2: Net-(U13-GND-Pad11) -> GND
- U12 pad 3: unconnected-(U13-CLKIN-Pad3) -> GND
- U12 pad 4: unconnected-(U13-SPEED-Pad4) -> Net-(U12-SPEED)
- U12 pad 5: Net-(U13-CAP-Pad5) -> Net-(C48-Pad2)
- U12 pad 6: Net-(U13-CAP-Pad5) -> Net-(C48-Pad1)
- U12 pad 7: unconnected-(U13-AINP-Pad7) -> Net-(J30-Pin_2)
- U12 pad 8: unconnected-(U13-AINN-Pad8) -> Net-(J30-Pin_1)
- U12 pad 9: unconnected-(U13-VREFN-Pad9) -> GND
