File: Alpha_Breakout.kicad_sch (KiCad schematic)
At the start: 0 parts

Commit message: Added Thermocouple Amp sheet
Other:
- added sheet thermoAmps (thermoAms.kicad_sch)
Changed lines of the file:
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@@
 		(exclude_from_sim no)
 		(at 42.418 27.178 0)
+		(effects
+			(font
+				(size 1.27 1.27)
+			)
+		)
 	)
 	(text "SebTEst\n"
@@
 		)
 	)
+	(sheet
+		(at 66.04 55.88)
+		(size 40.64 11.43)
+		(exclude_from_sim no)
+		(in_bom yes)
+		(on_board yes)
+		(dnp no)
+		(fields_autoplaced yes)
+		(stroke
+			(width 0.1524)
+			(type solid)
+		)
+		(fill
+			(color 0 0 0 0.0000)
+		)
+		(property "Sheetname" "thermoAmps"
+			(at 66.04 55.1684 0)
+			(effects
+				(font
+					(size 1.27 1.27)
+				)
+				(justify left bottom)
+			)
+		)
+		(property "Sheetfile" "thermoAms.kicad_sch"
+			(at 66.04 67.8946 0)
+			(effects
+				(font
+					(size 1.27 1.27)
+				)
+				(justify left top)
+			)
+		)
+		(instances
+			(project "Alpha_Breakout"
+				(path "/bb73515c-a1ce-4448-8899-3a433fb04c26"
+					(page "5")
+				)
+			)
+		)
+	)

Commit message: power
Other:
- added sheet Power (Power.kicad_sch)
- sheet stm32f1 ports: added SPI1_MISO, SPI1_MOSI, SPI1_SCK; removed none
- note removed: "Luke"
- note removed: "SebTEst"
Changed lines of the file:
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@@
 		(title "Alpha_Peripheral_Board")
-	)
-	(text "Luke\n"
-		(exclude_from_sim no)
-		(at 42.418 27.178 0)
-		(effects
-			(font
-				(size 1.27 1.27)
-			)
-		)
-	)
-	(text "SebTEst\n"
-		(exclude_from_sim no)
-		(at 25.4 180.594 0)
-		(effects
-			(font
-				(size 1.27 1.27)
-			)
-		)
 	)
 	(wire
@@
 	)
 	(sheet
-		(at 140.97 88.9)
-		(size 25.4 12.7)
+		(at 140.97 76.2)
+		(size 25.4 25.4)
 		(exclude_from_sim no)
 		(in_bom yes)
@@
 		)
 		(property "Sheetname" "stm32f1"
-			(at 140.97 88.1884 0)
+			(at 140.97 75.4884 0)
 			(effects
 				(font
@@
 			)
 		)
+		(pin "SPI1_SCK" input
+			(at 140.97 81.28 180)
+			(effects
+				(font
+					(size 1.27 1.27)
+				)
+				(justify left)
+			)
+		)
+		(pin "SPI1_MOSI" input
+			(at 140.97 83.82 180)
+			(effects
+				(font
+					(size 1.27 1.27)
+				)
+				(justify left)
+			)
+		)
+		(pin "SPI1_MISO" input
+			(at 140.97 86.36 180)
+			(effects
+				(font
+					(size 1.27 1.27)
+				)
+				(justify left)
+			)
+		)
 		(instances
 			(project "Alpha_Breakout"
@@
 				)
 			)
+		)
+	)
+	(sheet
+		(at 100.33 121.92)
+		(size 27.94 17.78)
+		(exclude_from_sim no)
+		(in_bom yes)
+		(on_board yes)
+		(dnp no)
+		(fields_autoplaced yes)
+		(stroke
+			(width 0.1524)
+			(type solid)
+		)
+		(fill
+			(color 0 0 0 0.0000)
+		)
+		(property "Sheetname" "Power"
+			(at 100.33 121.2084 0)
+			(effects
+				(font
+					(size 1.27 1.27)
+				)
+				(justify left bottom)
+			)
+		)
+		(property "Sheetfile" "Power.kicad_sch"
+			(at 100.33 140.2846 0)
+			(effects
+				(font
+					(size 1.27 1.27)
+				)
+				(justify left top)
+			)
+		)
+		(instances
+			(project "Alpha_Breakout"
+				(path "/bb73515c-a1ce-4448-8899-3a433fb04c26"
+					(page "6")
+				)
+			)

Commit message: reg🟡
Other:
- sheet stm32f1 ports: added TC1_CS, TC2_CS, TC3_CS, TC4_CS; removed none
Changed lines of the file:
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@@
 	)
 	(sheet
-		(at 66.04 55.88)
-		(size 40.64 11.43)
+		(at 99.06 53.34)
+		(size 22.86 19.05)
 		(exclude_from_sim no)
 		(in_bom yes)
@@
 		)
 		(property "Sheetname" "thermoAmps"
-			(at 66.04 55.1684 0)
+			(at 99.06 52.6284 0)
 			(effects
 				(font
@@
 		)
 		(property "Sheetfile" "thermoAms.kicad_sch"
-			(at 66.04 67.8946 0)
+			(at 99.06 72.9746 0)
 			(effects
 				(font
@@
 	)
 	(sheet
-		(at 140.97 76.2)
-		(size 25.4 25.4)
+		(at 140.97 63.5)
+		(size 25.4 38.1)
 		(exclude_from_sim no)
 		(in_bom yes)
@@
 		)
 		(property "Sheetname" "stm32f1"
-			(at 140.97 75.4884 0)
+			(at 140.97 62.7884 0)
 			(effects
 				(font
@@
 		)
 		(pin "SPI1_SCK" input
+			(at 140.97 76.2 180)
+			(effects
+				(font
+					(size 1.27 1.27)
+				)
+				(justify left)
+			)
+		)
+		(pin "SPI1_MOSI" input
+			(at 140.97 78.74 180)
+			(effects
+				(font
+					(size 1.27 1.27)
+				)
+				(justify left)
+			)
+		)
+		(pin "SPI1_MISO" input
 			(at 140.97 81.28 180)
 			(effects
@@
 			)
 		)
-		(pin "SPI1_MOSI" input
-			(at 140.97 83.82 180)
+		(pin "TC2_CS" input
+			(at 140.97 71.12 180)
 			(effects
 				(font
@@
 			)
 		)
-		(pin "SPI1_MISO" input
-			(at 140.97 86.36 180)
+		(pin "TC4_CS" input
+			(at 140.97 66.04 180)
 			(effects
 				(font
+					(size 1.27 1.27)
+				)
+				(justify left)
+			)
+		)
+		(pin "TC3_CS" input
+			(at 140.97 68.58 180)
+			(effects
+				(font
+					(size 1.27 1.27)
+				)
+				(justify left)
+			)
+		)
+		(pin "TC1_CS" input
+			(at 140.97 73.66 180)
+			(effects
+				(font

Commit message: Routed ThermoAmps to STM32
Other:
- sheet thermoAmps ports: added SPI1_MISO, SPI1_MOSI, SPI1_SCK, TC1_CS, TC2_CS, TC3_CS, TC4_CS; removed none

Commit message: plug🔌
Other:
- added sheet Accelerometer (Accelerometer.kicad_sch)
- added sheet RS-485 (RS-485.kicad_sch)
- sheet stm32f1 ports: added DIR_RS485, I2C1_SCL, I2C1_SDA, I2C2_SCL, I2C2_SDA, UART_2_RX, UART_2_TX; removed SCL, SDA

Commit message: Added Solenoids (Double Check Diode Type?)
Other:
- added sheet Solenoids (Solenoids.kicad_sch)
Changed lines of the file:
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@@
+	)
+	(sheet
+		(at 57.15 142.24)
+		(size 31.75 26.67)
+		(exclude_from_sim no)
+		(in_bom yes)
+		(on_board yes)
+		(dnp no)
+		(fields_autoplaced yes)
+		(stroke
+			(width 0.1524)
+			(type solid)
+		)
+		(fill
+			(color 0 0 0 0.0000)
+		)
+		(property "Sheetname" "Solenoids"
+			(at 57.15 141.5284 0)
+			(effects
+				(font
+					(size 1.27 1.27)
+				)
+				(justify left bottom)
+			)
+		)
+		(property "Sheetfile" "Solenoids.kicad_sch"
+			(at 57.15 169.4946 0)
+			(effects
+				(font
+					(size 1.27 1.27)
+				)
+				(justify left top)
+			)
+		)
+		(instances
+			(project "Alpha_Breakout"
+				(path "/bb73515c-a1ce-4448-8899-3a433fb04c26"
+					(page "9")
+				)
+			)
+		)
 	)
 	(sheet

Commit message: oops I forgot to specify resistor footprint
Other:
- sheet Solenoids ports: added S1, S2, S3, S4; removed none
Changed lines of the file:
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@@
 	)
 	(sheet
-		(at 57.15 142.24)
+		(at 49.53 92.71)
 		(size 31.75 26.67)
 		(exclude_from_sim no)
@@
 		)
 		(property "Sheetname" "Solenoids"
-			(at 57.15 141.5284 0)
+			(at 49.53 91.9984 0)
 			(effects
 				(font
@@
 		)
 		(property "Sheetfile" "Solenoids.kicad_sch"
-			(at 57.15 169.4946 0)
+			(at 49.53 119.9646 0)
 			(effects
 				(font
@@
 			)
 		)
+		(pin "S1" input
+			(at 66.04 92.71 90)
+			(effects
+				(font
+					(size 1.27 1.27)
+				)
+				(justify right)
+			)
+		)
+		(pin "S2" input
+			(at 68.58 92.71 90)
+			(effects
+				(font
+					(size 1.27 1.27)
+				)
+				(justify right)
+			)
+		)
+		(pin "S3" input
+			(at 71.12 92.71 90)
+			(effects
+				(font
+					(size 1.27 1.27)
+				)
+				(justify right)
+			)
+		)
+		(pin "S4" input
+			(at 73.66 92.71 90)
+			(effects
+				(font
+					(size 1.27 1.27)
+				)
+				(justify right)
+			)
+		)

Commit message: Connected solenoids, some error fixes
Other:
- sheet stm32f1 ports: added S1, S2, S3, S4; removed none
Changed lines of the file:
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@@
+	(wire
+		(pts
+			(xy 127 88.9) (xy 140.97 88.9)
+		)
+		(stroke
+			(width 0)
+			(type default)
+		)
+	)
 	(wire
 		(pts
@@
 	(wire
 		(pts
-			(xy 116.84 105.41) (xy 116.84 92.71)
+			(xy 127 86.36) (xy 140.97 86.36)
+		)
+		(stroke
+			(width 0)
+			(type default)
+		)
+	)
+	(wire
+		(pts
+			(xy 116.84 135.89) (xy 116.84 97.79)
 		)
 		(stroke
@@
 	(wire
 		(pts
-			(xy 109.22 105.41) (xy 116.84 105.41)
+			(xy 110.49 135.89) (xy 116.84 135.89)
 		)
 		(stroke
@@
 	(wire
 		(pts
-			(xy 118.11 107.95) (xy 118.11 95.25)
+			(xy 118.11 138.43) (xy 118.11 100.33)
 		)
 		(stroke
@@
 	(wire
 		(pts
-			(xy 118.11 95.25) (xy 140.97 95.25)
+			(xy 118.11 100.33) (xy 140.97 100.33)
 		)
 		(stroke
@@
 	(wire
 		(pts
-			(xy 116.84 92.71) (xy 140.97 92.71)
-		)
-		(stroke
-			(width 0)
-			(type default)
-		)
-	)
-	(wire
-		(pts
-			(xy 109.22 107.95) (xy 118.11 107.95)
+			(xy 116.84 97.79) (xy 140.97 97.79)
+		)
+		(stroke
+			(width 0)
+			(type default)
+		)
+	)
+	(wire
+		(pts
+			(xy 110.49 138.43) (xy 118.11 138.43)
 		)
 		(stroke
@@
 	(wire
 		(pts
+			(xy 127 93.98) (xy 140.97 93.98)
+		)
+		(stroke
+			(width 0)
+			(type default)
+		)
+	)
+	(wire
+		(pts
 			(xy 114.3 81.28) (xy 140.97 81.28)
+		)
+		(stroke
+			(width 0)
+			(type default)
+		)
+	)
+	(wire
+		(pts
+			(xy 127 91.44) (xy 140.97 91.44)
 		)
 		(stroke
@@
 	)
 	(sheet
-		(at 49.53 92.71)
-		(size 31.75 26.67)
+		(at 102.87 83.82)
+		(size 24.13 11.43)
 		(exclude_from_sim no)
 		(in_bom yes)
@@
 		)
 		(property "Sheetname" "Solenoids"
-			(at 49.53 91.9984 0)
+			(at 102.87 83.1084 0)
 			(effects
 				(font
@@
 		)
 		(property "Sheetfile" "Solenoids.kicad_sch"
-			(at 49.53 119.9646 0)
+			(at 102.87 95.8346 0)
 			(effects
 				(font
@@
 		)
 		(pin "S1" input
-			(at 66.04 92.71 90)
+			(at 127 86.36 0)
 			(effects
 				(font
@@
 		)
 		(pin "S2" input
-			(at 68.58 92.71 90)
+			(at 127 88.9 0)
 			(effects
 				(font
@@
 		)
 		(pin "S3" input
-			(at 71.12 92.71 90)
+			(at 127 91.44 0)
 			(effects
 				(font
@@
 		)
 		(pin "S4" input
-			(at 73.66 92.71 90)
+			(at 127 93.98 0)
 			(effects
 				(font
@@
 	(sheet
 		(at 140.97 63.5)
-		(size 25.4 38.1)
+		(size 25.4 44.45)
 		(exclude_from_sim no)
 		(in_bom yes)
@@
 		)
 		(property "Sheetfile" "stm32f1.kicad_sch"
-			(at 140.97 102.1846 0)
+			(at 140.97 108.5346 0)
 			(effects
 				(font
@@
 		)
 		(pin "I2C1_SCL" input
-			(at 140.97 92.71 180)
+			(at 140.97 97.79 180)
 			(effects
 				(font
@@
 		)
 		(pin "I2C1_SDA" input
-			(at 140.97 95.25 180)
+			(at 140.97 100.33 180)
 			(effects
 				(font
@@
 				)
 				(justify right)
+			)
+		)
+		(pin "S2" input
+			(at 140.97 88.9 180)
+			(effects
+				(font
+					(size 1.27 1.27)
+				)
+				(justify left)
+			)
+		)
+		(pin "S1" input
+			(at 140.97 86.36 180)
+			(effects
+				(font
+					(size 1.27 1.27)
+				)
+				(justify left)
+			)
+		)
+		(pin "S3" input
+			(at 140.97 91.44 180)
+			(effects
+				(font
+					(size 1.27 1.27)
+				)
+				(justify left)
+			)
+		)
+		(pin "S4" input
+			(at 140.97 93.98 180)
+			(effects
+				(font
+					(size 1.27 1.27)
+				)
+				(justify left)
 			)
 		)
@@
 	)
 	(sheet
-		(at 85.09 102.87)
+		(at 86.36 133.35)
 		(size 24.13 7.62)
 		(exclude_from_sim no)
@@
 		)
 		(property "Sheetname" "ADCs"
-			(at 85.09 102.1584 0)
+			(at 86.36 132.6384 0)
 			(effects
 				(font
@@
 		)
 		(property "Sheetfile" "ADCs.kicad_sch"
-			(at 85.09 111.0746 0)
+			(at 86.36 141.5546 0)
 			(effects
 				(font
@@
 		)
 		(pin "SCL" input
-			(at 109.22 105.41 0)
+			(at 110.49 135.89 0)
 			(effects
 				(font
@@
 		)
 		(pin "SDA" input
-			(at 109.22 107.95 0)
+			(at 110.49 138.43 0)
 			(effects
 				(font
@@
 	)
 	(sheet
-		(at 100.33 121.92)
+		(at 142.24 123.19)
 		(size 27.94 17.78)
 		(exclude_from_sim no)
@@
 		)
 		(property "Sheetname" "Power"
-			(at 100.33 121.2084 0)
+			(at 142.24 122.4784 0)
 			(effects
 				(font
@@
 		)
 		(property "Sheetfile" "Power.kicad_sch"
-			(at 100.33 140.2846 0)
-			(effects
-				(font
+			(at 142.24 141.5546 0)
+			(effects
+				(font
