File: Alpha_Breakout.kicad_sch (KiCad schematic)
At the start: 0 parts

Commit message: read description
Other:
- added sheet ADS1231 (ADS1231.kicad_sch)
Changed lines of the file:
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@@
 	(wire
 		(pts
-			(xy 127 88.9) (xy 140.97 88.9)
+			(xy 110.49 88.9) (xy 140.97 88.9)
 		)
 		(stroke
@@
 	(wire
 		(pts
-			(xy 127 86.36) (xy 140.97 86.36)
-		)
-		(stroke
-			(width 0)
-			(type default)
-		)
-	)
-	(wire
-		(pts
-			(xy 116.84 135.89) (xy 116.84 97.79)
+			(xy 110.49 86.36) (xy 140.97 86.36)
+		)
+		(stroke
+			(width 0)
+			(type default)
+		)
+	)
+	(wire
+		(pts
+			(xy 133.35 109.22) (xy 133.35 97.79)
 		)
 		(stroke
@@
 	(wire
 		(pts
-			(xy 110.49 135.89) (xy 116.84 135.89)
+			(xy 111.76 109.22) (xy 133.35 109.22)
 		)
 		(stroke
@@
 	(wire
 		(pts
-			(xy 118.11 138.43) (xy 118.11 100.33)
+			(xy 135.89 111.76) (xy 135.89 100.33)
 		)
 		(stroke
@@
 	(wire
 		(pts
-			(xy 118.11 100.33) (xy 140.97 100.33)
+			(xy 135.89 100.33) (xy 140.97 100.33)
 		)
 		(stroke
@@
 	(wire
 		(pts
-			(xy 116.84 97.79) (xy 140.97 97.79)
-		)
-		(stroke
-			(width 0)
-			(type default)
-		)
-	)
-	(wire
-		(pts
-			(xy 110.49 138.43) (xy 118.11 138.43)
+			(xy 133.35 97.79) (xy 140.97 97.79)
+		)
+		(stroke
+			(width 0)
+			(type default)
+		)
+	)
+	(wire
+		(pts
+			(xy 111.76 111.76) (xy 135.89 111.76)
 		)
 		(stroke
@@
 	(wire
 		(pts
-			(xy 127 93.98) (xy 140.97 93.98)
+			(xy 110.49 93.98) (xy 140.97 93.98)
 		)
 		(stroke
@@
 	(wire
 		(pts
-			(xy 127 91.44) (xy 140.97 91.44)
+			(xy 110.49 91.44) (xy 140.97 91.44)
 		)
 		(stroke
@@
 	)
 	(sheet
-		(at 102.87 83.82)
+		(at 86.36 83.82)
 		(size 24.13 11.43)
 		(exclude_from_sim no)
@@
 		)
 		(property "Sheetname" "Solenoids"
-			(at 102.87 83.1084 0)
+			(at 86.36 83.1084 0)
 			(effects
 				(font
@@
 		)
 		(property "Sheetfile" "Solenoids.kicad_sch"
-			(at 102.87 95.8346 0)
+			(at 86.36 95.8346 0)
 			(effects
 				(font
@@
 		)
 		(pin "S1" input
-			(at 127 86.36 0)
+			(at 110.49 86.36 0)
 			(effects
 				(font
@@
 		)
 		(pin "S2" input
-			(at 127 88.9 0)
+			(at 110.49 88.9 0)
 			(effects
 				(font
@@
 		)
 		(pin "S3" input
-			(at 127 91.44 0)
+			(at 110.49 91.44 0)
 			(effects
 				(font
@@
 		)
 		(pin "S4" input
-			(at 127 93.98 0)
+			(at 110.49 93.98 0)
 			(effects
 				(font
@@
 	)
 	(sheet
+		(at 143.51 31.75)
+		(size 20.32 16.51)
+		(exclude_from_sim no)
+		(in_bom yes)
+		(on_board yes)
+		(dnp no)
+		(fields_autoplaced yes)
+		(stroke
+			(width 0.1524)
+			(type solid)
+		)
+		(fill
+			(color 0 0 0 0.0000)
+		)
+		(property "Sheetname" "ADS1231"
+			(at 143.51 31.0384 0)
+			(effects
+				(font
+					(size 1.27 1.27)
+				)
+				(justify left bottom)
+			)
+		)
+		(property "Sheetfile" "ADS1231.kicad_sch"
+			(at 143.51 48.8446 0)
+			(effects
+				(font
+					(size 1.27 1.27)
+				)
+				(justify left top)
+			)
+		)
+		(instances
+			(project "Alpha_Breakout"
+				(path "/bb73515c-a1ce-4448-8899-3a433fb04c26"
+					(page "10")
+				)
+			)
+		)
+	)
+	(sheet
 		(at 140.97 63.5)
 		(size 25.4 44.45)
@@
 	)
 	(sheet
-		(at 86.36 133.35)
-		(size 24.13 7.62)
+		(at 97.79 106.68)
+		(size 13.97 8.89)
 		(exclude_from_sim no)
 		(in_bom yes)
@@
 		)
 		(property "Sheetname" "ADCs"
-			(at 86.36 132.6384 0)
+			(at 97.79 105.9684 0)
 			(effects
 				(font
@@
 		)
 		(property "Sheetfile" "ADCs.kicad_sch"
-			(at 86.36 141.5546 0)
+			(at 97.79 116.1546 0)
 			(effects
 				(font
@@
 		)
 		(pin "SCL" input
-			(at 110.49 135.89 0)
+			(at 111.76 109.22 0)
 			(effects
 				(font
@@
 		)
 		(pin "SDA" input
-			(at 110.49 138.43 0)
+			(at 111.76 111.76 0)
 			(effects
 				(font
@@
 	)
 	(sheet
-		(at 142.24 123.19)
+		(at 138.43 125.73)
 		(size 27.94 17.78)
 		(exclude_from_sim no)
@@
 		)
 		(property "Sheetname" "Power"
-			(at 142.24 122.4784 0)
+			(at 138.43 125.0184 0)
 			(effects
 				(font
@@
 		)
 		(property "Sheetfile" "Power.kicad_sch"
-			(at 142.24 141.5546 0)
-			(effects
-				(font
+			(at 138.43 144.0946 0)
+			(effects
+				(font

Commit message: arranged board
Other:
- added sheet Hardware_Safe (Hardware_Safe.kicad_sch)
- added sheet Pyro (Pyro.kicad_sch)
- sheet stm32f1 ports: added BW1, K1, K2, PYRO1; removed none
Changed lines of the file:
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@@
+	(wire
+		(pts
+			(xy 151.13 132.08) (xy 132.08 132.08)
+		)
+		(stroke
+			(width 0)
+			(type default)
+		)
+	)
 	(wire
 		(pts
@@
 	(wire
 		(pts
+			(xy 151.13 107.95) (xy 151.13 132.08)
+		)
+		(stroke
+			(width 0)
+			(type default)
+		)
+	)
+	(wire
+		(pts
 			(xy 116.84 78.74) (xy 140.97 78.74)
 		)
@@
 	(wire
 		(pts
+			(xy 148.59 129.54) (xy 132.08 129.54)
+		)
+		(stroke
+			(width 0)
+			(type default)
+		)
+	)
+	(wire
+		(pts
 			(xy 166.37 71.12) (xy 179.07 71.12)
 		)
@@
 	(wire
 		(pts
+			(xy 175.26 129.54) (xy 158.75 129.54)
+		)
+		(stroke
+			(width 0)
+			(type default)
+		)
+	)
+	(wire
+		(pts
 			(xy 166.37 66.04) (xy 173.99 66.04)
 		)
@@
 	(wire
 		(pts
+			(xy 158.75 129.54) (xy 158.75 107.95)
+		)
+		(stroke
+			(width 0)
+			(type default)
+		)
+	)
+	(wire
+		(pts
 			(xy 127 59.69) (xy 127 68.58)
 		)
@@
 	(wire
 		(pts
+			(xy 148.59 107.95) (xy 148.59 129.54)
+		)
+		(stroke
+			(width 0)
+			(type default)
+		)
+	)
+	(wire
+		(pts
+			(xy 146.05 127) (xy 132.08 127)
+		)
+		(stroke
+			(width 0)
+			(type default)
+		)
+	)
+	(wire
+		(pts
 			(xy 179.07 71.12) (xy 179.07 62.23)
 		)
@@
 	(wire
 		(pts
+			(xy 146.05 107.95) (xy 146.05 127)
+		)
+		(stroke
+			(width 0)
+			(type default)
+		)
+	)
+	(wire
+		(pts
 			(xy 114.3 81.28) (xy 140.97 81.28)
 		)
@@
 			(width 0)
 			(type default)
+		)
+	)
+	(sheet
+		(at 115.57 124.46)
+		(size 16.51 10.16)
+		(exclude_from_sim no)
+		(in_bom yes)
+		(on_board yes)
+		(dnp no)
+		(fields_autoplaced yes)
+		(stroke
+			(width 0.1524)
+			(type solid)
+		)
+		(fill
+			(color 0 0 0 0.0000)
+		)
+		(property "Sheetname" "Hardware_Safe"
+			(at 115.57 123.7484 0)
+			(effects
+				(font
+					(size 1.27 1.27)
+				)
+				(justify left bottom)
+			)
+		)
+		(property "Sheetfile" "Hardware_Safe.kicad_sch"
+			(at 115.57 135.2046 0)
+			(effects
+				(font
+					(size 1.27 1.27)
+				)
+				(justify left top)
+			)
+		)
+		(pin "K1" input
+			(at 132.08 127 0)
+			(effects
+				(font
+					(size 1.27 1.27)
+				)
+				(justify right)
+			)
+		)
+		(pin "BW1" input
+			(at 132.08 132.08 0)
+			(effects
+				(font
+					(size 1.27 1.27)
+				)
+				(justify right)
+			)
+		)
+		(pin "K2" input
+			(at 132.08 129.54 0)
+			(effects
+				(font
+					(size 1.27 1.27)
+				)
+				(justify right)
+			)
+		)
+		(instances
+			(project "Alpha_Breakout"
+				(path "/bb73515c-a1ce-4448-8899-3a433fb04c26"
+					(page "11")
+				)
+			)
 		)
 	)
@@
 	)
 	(sheet
-		(at 143.51 31.75)
+		(at 143.51 35.56)
 		(size 20.32 16.51)
 		(exclude_from_sim no)
@@
 		)
 		(property "Sheetname" "ADS1231"
-			(at 143.51 31.0384 0)
+			(at 143.51 34.8484 0)
 			(effects
 				(font
@@
 		)
 		(property "Sheetfile" "ADS1231.kicad_sch"
-			(at 143.51 48.8446 0)
+			(at 143.51 52.6546 0)
 			(effects
 				(font
@@
 				(path "/bb73515c-a1ce-4448-8899-3a433fb04c26"
 					(page "10")
+				)
+			)
+		)
+	)
+	(sheet
+		(at 175.26 125.73)
+		(size 13.97 7.62)
+		(exclude_from_sim no)
+		(in_bom yes)
+		(on_board yes)
+		(dnp no)
+		(fields_autoplaced yes)
+		(stroke
+			(width 0.1524)
+			(type solid)
+		)
+		(fill
+			(color 0 0 0 0.0000)
+		)
+		(property "Sheetname" "Pyro"
+			(at 175.26 125.0184 0)
+			(effects
+				(font
+					(size 1.27 1.27)
+				)
+				(justify left bottom)
+			)
+		)
+		(property "Sheetfile" "Pyro.kicad_sch"
+			(at 175.26 133.9346 0)
+			(effects
+				(font
+					(size 1.27 1.27)
+				)
+				(justify left top)
+			)
+		)
+		(pin "PYRO1" input
+			(at 175.26 129.54 180)
+			(effects
+				(font
+					(size 1.27 1.27)
+				)
+				(justify left)
+			)
+		)
+		(instances
+			(project "Alpha_Breakout"
+				(path "/bb73515c-a1ce-4448-8899-3a433fb04c26"
+					(page "12")
 				)
 			)
@@
 		(on_board yes)
 		(dnp no)
-		(fields_autoplaced yes)
 		(stroke
 			(width 0.1524)
@@
 		)
 		(property "Sheetfile" "stm32f1.kicad_sch"
-			(at 140.97 108.5346 0)
+			(at 140.462 108.966 0)
 			(effects
 				(font
@@
 		(pin "S4" input
 			(at 140.97 93.98 180)
+			(effects
+				(font
+					(size 1.27 1.27)
+				)
+				(justify left)
+			)
+		)
+		(pin "BW1" input
+			(at 151.13 107.95 270)
+			(effects
+				(font
+					(size 1.27 1.27)
+				)
+				(justify left)
+			)
+		)
+		(pin "K1" input
+			(at 146.05 107.95 270)
+			(effects
+				(font
+					(size 1.27 1.27)
+				)
+				(justify left)
+			)
+		)
+		(pin "K2" input
+			(at 148.59 107.95 270)
+			(effects
+				(font
+					(size 1.27 1.27)
+				)
+				(justify left)
+			)
+		)
+		(pin "PYRO1" input
+			(at 158.75 107.95 270)
 			(effects
 				(font
@@
 	)
 	(sheet
-		(at 138.43 125.73)
+		(at 227.33 123.19)
 		(size 27.94 17.78)
 		(exclude_from_sim no)
@@
 		)
 		(property "Sheetname" "Power"
-			(at 138.43 125.0184 0)
+			(at 227.33 122.4784 0)
 			(effects
 				(font
@@
 		)
 		(property "Sheetfile" "Power.kicad_sch"
-			(at 138.43 144.0946 0)
-			(effects
-				(font
+			(at 227.33 141.5546 0)
+			(effects
+				(font

Commit message: Breakout
Other:
- added sheet Breakout (breakout.kicad_sch)
- sheet ADS1231 ports: added LC_DRDY/DOUT, LC_SCLK; removed none
- sheet stm32f1 ports: added LC_DRDY/DOUT, LC_SCLK, PA13, PA14, PA15, PB3, PB4, PB5, PB8, PB9, PC13, PC14, PC15; removed none

Commit message: lots🅿️
Other:
- sheet Breakout ports: added none; removed PC13, PC14, PC15
- sheet stm32f1 ports: added none; removed PC13, PC14, PC15

Commit message: touchups 💅
Other:
- sheet Hardware_Safe ports: added none; removed K2
- sheet stm32f1 ports: added none; removed K2
Changed lines of the file:
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@@
 	(wire
 		(pts
-			(xy 135.89 129.54) (xy 115.57 129.54)
+			(xy 133.35 125.73) (xy 118.11 125.73)
 		)
 		(stroke
@@
 	(wire
 		(pts
-			(xy 135.89 115.57) (xy 135.89 129.54)
+			(xy 133.35 115.57) (xy 133.35 125.73)
 		)
 		(stroke
@@
 	(wire
 		(pts
-			(xy 133.35 115.57) (xy 133.35 127)
-		)
-		(stroke
-			(width 0)
-			(type default)
-		)
-	)
-	(wire
-		(pts
-			(xy 130.81 115.57) (xy 130.81 124.46)
+			(xy 130.81 115.57) (xy 130.81 123.19)
 		)
 		(stroke
@@
 	(wire
 		(pts
-			(xy 133.35 127) (xy 115.57 127)
-		)
-		(stroke
-			(width 0)
-			(type default)
-		)
-	)
-	(wire
-		(pts
 			(xy 173.99 69.85) (xy 154.94 69.85)
 		)
@@
 	(wire
 		(pts
-			(xy 130.81 124.46) (xy 115.57 124.46)
+			(xy 130.81 123.19) (xy 118.11 123.19)
 		)
 		(stroke
@@
 	)
 	(sheet
-		(at 99.06 121.92)
-		(size 16.51 10.16)
+		(at 101.6 120.65)
+		(size 16.51 7.62)
 		(exclude_from_sim no)
 		(in_bom yes)
@@
 		)
 		(property "Sheetname" "Hardware_Safe"
-			(at 99.06 121.2084 0)
+			(at 101.6 119.9384 0)
 			(effects
 				(font
@@
 		)
 		(property "Sheetfile" "Hardware_Safe.kicad_sch"
-			(at 99.06 132.6646 0)
+			(at 101.6 128.8546 0)
 			(effects
 				(font
@@
 		)
 		(pin "K1" input
-			(at 115.57 124.46 0)
+			(at 118.11 123.19 0)
 			(effects
 				(font
@@
 		)
 		(pin "BW1" input
-			(at 115.57 129.54 0)
-			(effects
-				(font
-					(size 1.27 1.27)
-				)
-				(justify right)
-			)
-		)
-		(pin "K2" input
-			(at 115.57 127 0)
+			(at 118.11 125.73 0)
 			(effects
 				(font
@@
 		)
 		(pin "BW1" input
-			(at 135.89 115.57 270)
+			(at 133.35 115.57 270)
 			(effects
 				(font
@@
 			(effects
 				(font
-					(size 1.27 1.27)
-				)
-				(justify left)
-			)
-		)
-		(pin "K2" input
-			(at 133.35 115.57 270)
-			(effects
-				(font
