File: Power.kicad_sch (KiCad schematic)
At the start: 24 parts, among them J2 Conn_01x02, U5 AP63203WU

Commit message: reg🟡
Parts:
- added U7: LP2985-3.3, Package_TO_SOT_SMD:SOT-23-5, symbol Regulator_Linear:LP2985-3.3
- renumbered C16 to C15, C17 to C16, C27 to C17, C28 to C21, C21 to C22, C29 to C23, C22 to C24, C23 to C25, C30 to C26, C24 to C27, C25 to C28, C26 to C29, J2 to J3, L3 to L1, L4 to L2, PS2 to PS1, R15 to R10, R16 to R11, R13 to R8, R14 to R9, U5 to U6

Commit message: layout🏄‍♂️
Parts:
- added C30: 1uF, Capacitor_SMD:C_0402_1005Metric, symbol Device:C
- added C31: 2.2uF, Capacitor_SMD:C_0402_1005Metric, symbol Device:C
- added C32: 10nF, Capacitor_SMD:C_0402_1005Metric, symbol Device:C
- added IC1: LM66200DRLR, LM66200DRLR:SOT8, symbol LM66200DRLR:LM66200DRLR
- PS1: Description_1 Buck Switching Regulator IC Positive Fixed 5.15V 1 Output 12A 13-PowerVFQFN -> Buck Switching Regulator IC Positive Fixed 5.15V 1 Output 12A 13-PowerVFQFN
Connections:
- net +3.3V: no longer PS1.5 (MODE), PS1.6 (EN)
- net +5V: now also C17.1, U6.2 (EN), U6.3 (IN), IC1.2 (VOUT@1), IC1.7 (VOUT@2); no longer C20.1, C24.1, C27.1, C29.1, L1.2, R11.1
- net +BATT: now also U7.1 (VIN), U7.3 (ON/~{OFF}), C30.1; no longer C17.1, U6.2 (EN), U6.3 (IN)
- net GND: now also U7.2 (GND), C30.2, C31.2, C32.2, IC1.1 (GND@1), IC1.4 (ON), IC1.5 (GND@2)
- net at U7.4 (BP): now also C32.1
- net en: now reaches U7.5 (VOUT)
- net en: now also PS1.5 (MODE), PS1.6 (EN), C31.1
- new net BATT_V+: C20.1, C24.1, C27.1, C29.1, IC1.3 (VIN1), L1.2, R11.1
- new net USB_V+: IC1.6 (VIN2)
Other:
- note added: "Dual Diode"
- note added: "Enable Reg (3.3v)"
- moved on the sheet: C15, C16, C17, C18, C19, C20, C21, C22, C23, C24, C25, C26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

Commit message: fixed power
Parts:
- R11: value R -> 0
Connections:
- net FB: no longer C20.2, C24.2, C27.2, C29.2
- net GND: now also C20.2, C24.2, C27.2, C29.2
Changed lines of the file:
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@@
 	)
 	(junction
+		(at 181.61 139.7)
+		(diameter 0)
+		(color 0 0 0 0)
+	)
+	(junction
 		(at 168.91 116.84)
 		(diameter 0)
@@
 	)
 	(junction
-		(at 142.24 139.7)
-		(diameter 0)
-		(color 0 0 0 0)
-	)
-	(junction
-		(at 151.13 139.7)
-		(diameter 0)
-		(color 0 0 0 0)
-	)
-	(junction
 		(at 161.29 132.08)
 		(diameter 0)
@@
 	(wire
 		(pts
-			(xy 142.24 139.7) (xy 151.13 139.7)
-		)
-		(stroke
-			(width 0)
-			(type default)
-		)
-	)
-	(wire
-		(pts
 			(xy 124.46 67.31) (xy 113.03 67.31)
 		)
@@
 	)
 	(symbol
+		(lib_id "power:GND")
+		(at 181.61 139.7 0)
+		(unit 1)
+		(exclude_from_sim no)
+		(in_bom yes)
+		(on_board yes)
+		(dnp no)
+		(fields_autoplaced yes)
+		(property "Reference" "#PWR090"
+			(at 181.61 146.05 0)
+			(effects
+				(font
+					(size 1.27 1.27)
+				)
+				(hide yes)
+			)
+		)
+		(property "Value" "GND"
+			(at 181.61 144.78 0)
+			(effects
+				(font
+					(size 1.27 1.27)
+				)
+			)
+		)
+		(property "Footprint" ""
+			(at 181.61 139.7 0)
+			(effects
+				(font
+					(size 1.27 1.27)
+				)
+				(hide yes)
+			)
+		)
+		(property "Datasheet" ""
+			(at 181.61 139.7 0)
+			(effects
+				(font
+					(size 1.27 1.27)
+				)
+				(hide yes)
+			)
+		)
+		(property "Description" "Power symbol creates a global label with name \"GND\" , ground"
+			(at 181.61 139.7 0)
+			(effects
+				(font
+					(size 1.27 1.27)
+				)
+				(hide yes)
+			)
+		)
+		(pin "1"
+		)
+		(instances
+			(project "Alpha_Breakout"
+				(path "/bb73515c-a1ce-4448-8899-3a433fb04c26/f19b3af3-949e-4bd9-966f-10ca206af398"
+					(reference "#PWR090")
+					(unit 1)
+				)
+			)
+		)
+	)
+	(symbol
 		(lib_id "Device:R")
 		(at 142.24 135.89 0)
@@
 			)
 		)
-		(property "Value" "R"
+		(property "Value" "0"
 			(at 136.652 137.16 0)
 			(effects
