File: Power.kicad_sch (KiCad schematic)
At the start: 30 parts, among them IC1 LM66200DRLR, J3 Conn_01x02, U12 LM2576HVS-12, U6 AP63203WU, U7 LP2985-3.3

Commit message: oops I forgot to specify resistor footprint
Parts:
- removed U12: LM2576HVS-12, Package_TO_SOT_SMD:TO-263-5_TabPin3, symbol Regulator_Switching:LM2576HVS-12
Changed lines of the file:
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@@
-		)
-	)
-	(rectangle
-		(start 39.37 163.83)
-		(end 133.35 193.04)
-		(stroke
-			(width 0)
-			(type default)
-		)
-		(fill
-			(type none)
 		)
 	)
@@
 					(unit 1)
 				)
-			)
-		)
-	)
-	(symbol
-		(lib_id "Regulator_Switching:LM2576HVS-12")
-		(at 58.42 177.8 0)
-		(unit 1)
-		(exclude_from_sim no)
-		(in_bom yes)
-		(on_board yes)
-		(dnp no)
-		(fields_autoplaced yes)
-		(property "Reference" "U12"
-			(at 58.42 167.64 0)
-			(effects
-				(font
-					(size 1.27 1.27)
-				)
-			)
-		)
-		(property "Value" "LM2576HVS-12"
-			(at 58.42 170.18 0)
-			(effects
-				(font
-					(size 1.27 1.27)
-				)
-			)
-		)
-		(property "Footprint" "Package_TO_SOT_SMD:TO-263-5_TabPin3"
-			(at 58.42 184.15 0)
-			(effects
-				(font
-					(size 1.27 1.27)
-					(italic yes)
-				)
-				(justify left)
-				(hide yes)
-			)
-		)
-		(property "Datasheet" "http://www.ti.com/lit/ds/symlink/lm2576.pdf"
-			(at 58.42 177.8 0)
-			(effects
-				(font
-					(size 1.27 1.27)
-				)
-				(hide yes)
-			)
-		)
-		(property "Description" "12V, 3A SIMPLE SWITCHER® Step-Down Voltage Regulator, High Voltage Input, TO-263"
-			(at 58.42 177.8 0)
-			(effects
-				(font
-					(size 1.27 1.27)
-				)
-				(hide yes)
-			)
-		)
-		(pin "1"
-		)
-		(pin "3"
-		)
-		(pin "4"
-		)
-		(pin "5"
-		)
-		(pin "2"
-		)
-		(instances
-			(project ""
-				(path "/bb73515c-a1ce-4448-8899-3a433fb04c26/f19b3af3-949e-4bd9-966f-10ca206af398"
-					(reference "U12")
-					(unit 1)
-				)

Commit message: Added Power Status LEDs
Parts:
- added D5, D6, D7: LED, LED_SMD:LED_0603_1608Metric, symbol Device:LED
- added R18: 100, Resistor_SMD:R_0402_1005Metric, symbol Device:R
- added R19, R20: 200, Resistor_SMD:R_0402_1005Metric, symbol Device:R
Connections:
- net +3.3V: now also R18.1
- net +5V: now also R19.1
- net BATT_V+: now also R20.1
- net GND: now also D5.1 (K), D7.1 (K)
- net at IC1.8 (ST): now also D6.1 (K)
- new net: D7.2 (A), R20.2
- new net: D5.2 (A), R18.2
- new net: D6.2 (A), R19.2

Commit message: Not Entirely Sure
Parts:
- added D8: GREEN, LED_SMD:LED_0603_1608Metric, symbol Device:LED
- added R21: 200, Resistor_SMD:R_0402_1005Metric, symbol Device:R
- added TP1: TestPoint, TestPoint:TestPoint_Pad_D1.5mm, symbol Connector:TestPoint
- D6: value LED -> BLUE
Connections:
- net +5V: now also TP1.1
- net GND: now also D8.1 (K)
- net at D6.1 (K), IC1.8 (ST): now also R21.1
- new net: D8.2 (A), R21.2

Commit message: read description
Parts:
- added C48: 1uF, Capacitor_SMD:C_0402_1005Metric, symbol Device:C
- added U12: L78L10_SOT89, Package_TO_SOT_SMD:SOT-89-3, symbol Regulator_Linear:L78L10_SOT89
Connections:
- net +BATT: now also U12.3 (IN)
- net GND: now also C48.2, U12.2 (GND)
- new net +10V: C48.1, U12.1 (OUT)
Other:
- note added: "Load Cell Reg (10v)"
- moved on the sheet: C15, C16, C17, C18, C19, C20, C21, C22, C23, C24, C25, C26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

Commit message: Load Cell
Parts:
- removed C48: 1uF, Capacitor_SMD:C_0402_1005Metric, symbol Device:C
- removed U12: L78L10_SOT89, Package_TO_SOT_SMD:SOT-89-3, symbol Regulator_Linear:L78L10_SOT89
Other:
- note removed: "Load Cell Reg (10v)"

Commit message: added leds🔴🟡🔵
Parts:
- renumbered C15 to C30, C16 to C31, C17 to C32, C18 to C33, C19 to C34, C20 to C35, C21 to C36, C22 to C37, C23 to C38, C24 to C39, C25 to C40, C26 to C41, C27 to C42, C28 to C43, C29 to C44, C30 to C45, C31 to C46, C32 to C47, D5 to D1, D7 to D2, D6 to D3, D8 to D4, J3 to J22, R8 to R14, R9 to R15, R10 to R16, R11 to R17, R20 to R19, R19 to R20, TP1 to TP4, U7 to U10, U6 to U9

Commit message: done ✅
Parts:
- R15, R17: footprint (none) -> Resistor_SMD:R_0402_1005Metric
- TP4: footprint TestPoint:TestPoint_Pad_D1.5mm -> TestPoint:TestPoint_Pad_D1.0mm
Changed lines of the file:
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@@
 			)
 		)
-		(property "Footprint" ""
+		(property "Footprint" "Resistor_SMD:R_0402_1005Metric"
 			(at 115.062 143.51 90)
 			(effects
@@
 			)
 		)
-		(property "Footprint" "TestPoint:TestPoint_Pad_D1.5mm"
+		(property "Footprint" "TestPoint:TestPoint_Pad_D1.0mm"
 			(at 194.31 99.06 0)
 			(effects
@@
 			)
 		)
-		(property "Footprint" ""
+		(property "Footprint" "Resistor_SMD:R_0402_1005Metric"
 			(at 68.58 112.522 90)
 			(effects
