File: Alpha_Breakout.kicad_pcb (KiCad board)
At the start: 2 copper layers, 55.6 x 73.7 mm, 66 parts, among them IC1 LM66200DRLR, J1 USB_C_Receptacle_USB2.0_14P, J10 Conn_01x03, J11 Conn_01x03, J12 Conn_01x03, J13 Conn_01x03, J14 Conn_01x03, J15 Conn_01x03, J16 Conn_01x03, J17 Conn_01x03, J18 Conn_01x03, J19 Conn_01x03, J3 Conn_01x02, J4 Conn_01x03, J5 Conn_01x03, J6 Conn_01x03, J7 Conn_01x03, J8 Conn_01x03, J9 Conn_01x03, SW1 SW_Push, SW2 SW_Push, U1 STM32F103C8Tx, U2 CH340N, U3 ADS7828, U4 ADS7828, U5 MAX31856, U6 AP63203WU, U7 LP2985-3.3

Commit message: thermo🌡️
Parts:
- added C1: .01uF, Capacitor_SMD:C_0402_1005Metric, F.Cu at (147.0, 78.2)
- added C10: .01uF, Capacitor_SMD:C_0402_1005Metric, F.Cu at (147.3, 101.4)
- added C11: .01uF, Capacitor_SMD:C_0402_1005Metric, F.Cu at (146.3, 102.2)
- added C13: .01uF, Capacitor_SMD:C_0402_1005Metric, F.Cu at (156.0, 104.4)
- added C14: .01uF, Capacitor_SMD:C_0402_1005Metric, F.Cu at (156.0, 102.5)
- added C34: .01uF, Capacitor_SMD:C_0402_1005Metric, F.Cu at (138.5, 86.5)
- added C35: .01uF, Capacitor_SMD:C_0402_1005Metric, F.Cu at (140.4, 86.5)
- added C36: 0.1uF, Capacitor_SMD:C_0402_1005Metric, F.Cu at (139.4, 85.5)
- added C37: .01uF, Capacitor_SMD:C_0402_1005Metric, F.Cu at (139.3, 95.3)
- added C38: .01uF, Capacitor_SMD:C_0402_1005Metric, F.Cu at (137.4, 95.3)
- added C39: .01uF, Capacitor_SMD:C_0402_1005Metric, F.Cu at (145.6, 80.6)
- added C40: .01uF, Capacitor_SMD:C_0402_1005Metric, F.Cu at (162.1, 85.5)
- added C41: 0.1uF, Capacitor_SMD:C_0402_1005Metric, F.Cu at (146.6, 81.6)
- added C42: .01uF, Capacitor_SMD:C_0402_1005Metric, F.Cu at (155.3, 81.8)
- added C43: .01uF, Capacitor_SMD:C_0402_1005Metric, F.Cu at (155.3, 79.9)
- added C44: .01uF, Capacitor_SMD:C_0402_1005Metric, F.Cu at (164.7, 86.5)
- added C45: 0.1uF, Capacitor_SMD:C_0402_1005Metric, F.Cu at (162.8, 86.5)
- added C46: .01uF, Capacitor_SMD:C_0402_1005Metric, F.Cu at (164.2, 95.2)
- added C47: .01uF, Capacitor_SMD:C_0402_1005Metric, F.Cu at (162.3, 95.3)
- added J2: Conn_01x02, TerminalBlock_Phoenix:TerminalBlock_Phoenix_MPT-0,5-2-2.54_1x02_P2.54mm_Horizontal, F.Cu at (147.3, 64.9)
- added J20: Conn_01x02, TerminalBlock_Phoenix:TerminalBlock_Phoenix_MPT-0,5-2-2.54_1x02_P2.54mm_Horizontal, F.Cu at (138.3, 64.9)
- added J21: Conn_01x02, TerminalBlock_Phoenix:TerminalBlock_Phoenix_MPT-0,5-2-2.54_1x02_P2.54mm_Horizontal, F.Cu at (156.6, 64.9)
- added J22: Conn_01x02, TerminalBlock_Phoenix:TerminalBlock_Phoenix_MPT-0,5-2-2.54_1x02_P2.54mm_Horizontal, F.Cu at (165.6, 64.9)
- added R12: 100, Resistor_SMD:R_0402_1005Metric, F.Cu at (136.6, 86.5)
- added R13: 100, Resistor_SMD:R_0402_1005Metric, F.Cu at (141.8, 87.5)
- added R14: 100, Resistor_SMD:R_0402_1005Metric, F.Cu at (146.6, 83.4)
- added R15: 100, Resistor_SMD:R_0402_1005Metric, F.Cu at (146.6, 79.6)
- added R16: 100, Resistor_SMD:R_0402_1005Metric, F.Cu at (160.9, 86.5)
- added R17: 100, Resistor_SMD:R_0402_1005Metric, F.Cu at (164.0, 85.5)
- added R6: 100, Resistor_SMD:R_0402_1005Metric, F.Cu at (147.3, 105.2)
- added R7: 100, Resistor_SMD:R_0402_1005Metric, F.Cu at (147.3, 103.2)
- added U10: MAX31856, Package_SO:TSSOP-14_4.4x5mm_P0.65mm, F.Cu at (163.2, 90.9)
- added U8: MAX31856, Package_SO:TSSOP-14_4.4x5mm_P0.65mm, F.Cu at (138.9, 90.9)
- added U9: MAX31856, Package_SO:TSSOP-14_4.4x5mm_P0.65mm, F.Cu at (150.9, 81.1)
- C12: value .1uF -> 0.1uF
- moved C2 6.70 mm to (150.1, 85.7)
- moved C4 6.70 mm to (153.9, 86.8)
- moved C7 6.70 mm to (146.1, 95.4)
- moved U1 6.70 mm to (151.5, 92.4)
- moved C3 6.70 mm to (157.1, 94.8)
- moved C33 6.70 mm to (148.1, 96.9)
- moved C5 6.70 mm to (145.6, 89.7)
- moved R1 6.70 mm to (144.2, 92.2)
- moved R2 6.70 mm to (152.1, 85.7)
- moved R3 6.70 mm to (148.0, 87.6)
- moved C6 6.70 mm to (145.5, 93.1)
- moved C12 3.30 mm to (146.3, 104.0)
- moved U5 2.04 mm to (151.6, 102.9)
Connections:
- U5 pad 10: /thermoAmps/SPI1_SCK -> /stm32f1/SPI1_SCK
- U5 pad 11: /thermoAmps/SPI1_MISO -> /stm32f1/SPI1_MISO
- U5 pad 12: /thermoAmps/SPI1_MOSI -> /stm32f1/SPI1_MOSI
- U5 pad 9: /thermoAmps/TC4_CS -> /stm32f1/TC1_CS

Commit message: plug🔌
Parts:
- added J23: Conn_01x02, SM02B-GHS:CONN_SM02B-GHS_JST, F.Cu at (134.3, 63.9)
- added J24: Conn_01x04, SM04B-GHS:JST_SM04B-GHS-TB_LF__SN_-, F.Cu at (167.4, 52.8)
- added U11: SP3485EN, Package_SO:SOIC-8_3.9x4.9mm_P1.27mm, F.Cu at (140.3, 81.8)
- moved J20 3.90 mm to (142.2, 64.9)
- moved J22 3.56 mm to (162.1, 64.9)
- moved J2 1.50 mm to (148.8, 64.9)
- moved J21 1.16 mm to (155.5, 64.9)
Connections:
- C20 pad 2: FB -> GND
- C24 pad 2: FB -> GND
- C27 pad 2: FB -> GND
- C29 pad 2: FB -> GND
- C8 pad 2: +3.3V -> GND
- C9 pad 2: +3.3V -> GND
- U1 pad 10: unconnected-(U1-PA0-Pad10) -> /stm32f1/TC4_CS
- U1 pad 11: unconnected-(U1-PA1-Pad11) -> /stm32f1/TC3_CS
- U1 pad 12: unconnected-(U1-PA2-Pad12) -> /RS-485/TX_RS485
- U1 pad 13: /stm32f1/TC3_CS -> /RS-485/RX_RS485
- U1 pad 14: /stm32f1/TC4_CS -> /RS-485/DIR_RS485
- U1 pad 21: unconnected-(U1-PB10-Pad21) -> /Accelerometer/ACC_SDA
- U1 pad 22: unconnected-(U1-PB11-Pad22) -> /Accelerometer/ACC_SCL
Other:
- board text added: "RS-485"
- board text added: "TC1"
- board text added: "TC2"
- board text added: "TC3"
- board text added: "TC4"

Commit message: Added Solenoids (Double Check Diode Type?)
Parts:
- added Q1: CSD13381F4, CSD13381F4:DFN100X60X35-3N, F.Cu at (130.8, 57.5)
- added U12: LM2576HVS-12, Package_TO_SOT_SMD:TO-263-5_TabPin3, F.Cu at (139.6, 48.2)

Commit message: read description
Parts:
- removed J17, J19, J4, J5: Conn_01x03, TerminalBlock_Phoenix:TerminalBlock_Phoenix_MPT-0,5-3-2.54_1x03_P2.54mm_Horizontal
- added C48: 1uF, Capacitor_SMD:C_0402_1005Metric, F.Cu at (126.8, 117.3)
- added D1: D, Diode_SMD:D_SMA, F.Cu at (124.7, 71.9)
- added D2: D, Diode_SMD:D_SMA, F.Cu at (124.7, 78.9)
- added D3: D, Diode_SMD:D_SMA, F.Cu at (172.2, 78.2)
- added D4: D, Diode_SMD:D_SMA, F.Cu at (172.2, 71.1)
- added D5: LED, LED_SMD:LED_0603_1608Metric, F.Cu at (166.3, 119.1)
- added D6: BLUE, LED_SMD:LED_0603_1608Metric, F.Cu at (135.1, 119.0)
- added D7: LED, LED_SMD:LED_0603_1608Metric, F.Cu at (143.1, 120.2)
- added D8: GREEN, LED_SMD:LED_0603_1608Metric, F.Cu at (149.7, 120.3)
- added J25: Conn_01x02, TerminalBlock_Phoenix:TerminalBlock_Phoenix_MPT-0,5-2-2.54_1x02_P2.54mm_Horizontal, F.Cu at (119.2, 70.5)
- added J26: Conn_01x02, TerminalBlock_Phoenix:TerminalBlock_Phoenix_MPT-0,5-2-2.54_1x02_P2.54mm_Horizontal, F.Cu at (119.2, 77.1)
- added J27: Conn_01x02, TerminalBlock_Phoenix:TerminalBlock_Phoenix_MPT-0,5-2-2.54_1x02_P2.54mm_Horizontal, F.Cu at (177.6, 79.4)
- added J28: Conn_01x02, TerminalBlock_Phoenix:TerminalBlock_Phoenix_MPT-0,5-2-2.54_1x02_P2.54mm_Horizontal, F.Cu at (177.6, 72.8)
- added Q2: CSD13381F4, CSD13381F4:DFN100X60X35-3N, F.Cu at (127.0, 80.5)
- added Q3: CSD13381F4, CSD13381F4:DFN100X60X35-3N, F.Cu at (169.9, 79.9)
- added Q4: CSD13381F4, CSD13381F4:DFN100X60X35-3N, F.Cu at (169.9, 72.7)
- added R18: 100, Resistor_SMD:R_0402_1005Metric, F.Cu at (169.1, 118.3)
- added R19: 200, Resistor_SMD:R_0402_1005Metric, F.Cu at (136.3, 121.1)
- added R20: 200, Resistor_SMD:R_0402_1005Metric, F.Cu at (140.5, 120.5)
- added R21: 200, Resistor_SMD:R_0402_1005Metric, F.Cu at (152.3, 120.5)
- added U13: ADS1231ID, ADS1231ID:SOIC127P600X175-16N, F.Cu at (163.6, 86.9)
- U12: value LM2576HVS-12 -> L78L10_SOT89; footprint Package_TO_SOT_SMD:TO-263-5_TabPin3 -> Package_TO_SOT_SMD:SOT-89-3
- moved U12 73.1 mm to (128.2, 120.4)
- moved IC1 23.1 mm to (134.4, 121.1)
- moved C20 20.7 mm to (128.3, 125.2)
- moved C22 20.7 mm to (135.6, 127.6)
- moved R10 20.7 mm to (130.3, 134.5)
- moved C27 20.7 mm to (133.6, 131.1)
- moved PS1 20.7 mm to (130.3, 131.3)
- moved C15 20.7 mm to (127.8, 133.4)
- moved C16 20.7 mm to (127.8, 131.6)
- moved C18 20.7 mm to (133.3, 134.5)
- moved C19 20.7 mm to (130.9, 127.6)
- moved C24 20.7 mm to (133.0, 125.2)
- moved C25 20.7 mm to (126.3, 127.7)
- moved C29 20.7 mm to (126.2, 131.2)
- moved R8 20.7 mm to (127.8, 134.8)
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Connections:
- IC1 pad 8: unconnected-(IC1-ST-Pad8) -> Net-(D6-K)
- Q1 pad 1: unconnected-(Q1-Pad1) -> /Solenoids/S1
- Q1 pad 2: unconnected-(Q1-Pad2) -> GND
- Q1 pad 3: unconnected-(Q1-Pad3) -> Net-(D1-A)
- U1 pad 25: unconnected-(U1-PB12-Pad25) -> /Solenoids/S1
- U1 pad 26: unconnected-(U1-PB13-Pad26) -> /Solenoids/S2
- U1 pad 27: unconnected-(U1-PB14-Pad27) -> /Solenoids/S3
- U1 pad 28: unconnected-(U1-PB15-Pad28) -> /Solenoids/S4
- U10 pad 9: /stm32f1/TC1_CS -> /stm32f1/TC4_CS
- U12 pad 1: unconnected-(U12-VIN-Pad1) -> +10V
- U12 pad 2: unconnected-(U12-OUT-Pad2) -> GND
- U12 pad 3: unconnected-(U12-GND-Pad3) -> +BATT
- U5 pad 9: /stm32f1/TC1_CS -> /stm32f1/TC2_CS
- U8 pad 9: /stm32f1/TC1_CS -> /stm32f1/TC3_CS
Routing:
- net CH_00: track 36.9 -> 0.00 mm
- net CH_15: track 36.4 -> 0.00 mm
- net CH_07: track 30.5 -> 0.00 mm
- net CH_08: track 30.1 -> 0.00 mm
- net CH_01: track 28.5 -> 0.00 mm
- net CH_14: track 28.1 -> 0.00 mm
- net CH_06: track 22.1 -> 0.00 mm
- net CH_09: track 21.7 -> 0.00 mm
- net CH_02: track 20.1 -> 0.00 mm
- net CH_13: track 19.7 -> 0.00 mm
- net CH_05: track 14.6 -> 0.00 mm
- net CH_10: track 13.4 -> 0.00 mm
- net CH_12: track 11.7 -> 0.00 mm
- net CH_04: track 9.54 -> 0.00 mm
- net CH_11: track 8.50 -> 0.00 mm
Other:
- board size 55.6 x 73.7 mm -> 66.7 x 73.7 mm
- board text added: "ACCEL"

Commit message: arranged board
Parts:
- added J29: Conn_01x02, BM02B-GHS:JST_BM02B-GHS-TBT_LF__SN_, F.Cu at (128.1, 114.0)
- added J31: Conn_01x02, BM02B-GHS:JST_BM02B-GHS-TBT_LF__SN_, F.Cu at (135.6, 114.0)
- added J32: Conn_01x02, BM02B-GHS:JST_BM02B-GHS-TBT_LF__SN_, F.Cu at (165.2, 113.8)
Other:
- board text added: "BURN"
- board text added: "KEYS"

Commit message: estop added
Parts:
- added J33: Conn_01x02, BM02B-GHS:JST_BM02B-GHS-TBT_LF__SN_, F.Cu at (161.1, 114.2)
- added JP1: SolderJumper_2_Open, Jumper:SolderJumper-2_P1.3mm_Open_TrianglePad1.0x1.5mm, F.Cu at (155.3, 116.7)
- moved J32 3.41 mm to (168.6, 114.2)
Connections:
- D1 pad 1: +BATT -> SW_PWR
- D2 pad 1: +BATT -> SW_PWR
- D3 pad 1: +BATT -> SW_PWR
- D4 pad 1: +BATT -> SW_PWR
- J25 pad 1: +BATT -> SW_PWR
- J26 pad 1: +BATT -> SW_PWR
- J27 pad 1: +BATT -> SW_PWR
- J28 pad 1: +BATT -> SW_PWR
- U1 pad 20: unconnected-(U1-PB2-Pad20) -> +3.3V
- U1 pad 29: unconnected-(U1-PA8-Pad29) -> /Pyro/PYRO1
- U1 pad 5: unconnected-(U1-PD0-Pad5) -> +3.3V
- U1 pad 6: unconnected-(U1-PD1-Pad6) -> +3.3V
Other:
- board text added: "BYPASS"
- board text added: "ESTOP"
