File: Alpha_Breakout.kicad_pcb (KiCad board)
At the start: 2 copper layers, 66.7 x 74.4 mm, 163 parts, among them IC1 LM66200DRLR, J1 USB_C_Receptacle_USB2.0_14P, J10 Conn_01x03, J11 Conn_01x03, J12 Conn_01x03, J14 Conn_01x03, J15 Conn_01x03, J16 Conn_01x03, J18 Conn_01x02, J19 Conn_01x02, J20 Conn_01x02, J21 Conn_01x02, J22 Conn_01x02, J23 Conn_01x02, J24 Conn_01x04, J25 Conn_01x02, J26 Conn_01x02, J27 Conn_01x02, J28 Conn_01x02, J29 Conn_01x02, J3 Conn_01x03, J30 Conn_01x04, J31 Conn_01x02, J33 Conn_01x02, J34 Conn_01x02, J35 Conn_02x06_Odd_Even, J36 Conn_01x02, J4 Conn_01x03, J5 Conn_01x03, J7 Conn_01x03, J8 Conn_01x03, J9 Conn_01x03, Q1 CSD13381F4, Q2 CSD13381F4, Q3 CSD13381F4, Q4 CSD13381F4, Q5 SSM3J328R, Q6 L2N7002SLLT1G, SW1 SW_Push, SW2 SW_Push, U1 STM32F103C8Tx, U10 LP2985-3.3, U11 SP3485EN, U12 ADS1231ID, U12 L78L10_SOT89, U13 TCA9517ADGK, U2 CH340N, U3 ADS7828, U4 ADS7828, U5 MAX31856, U6 MAX31856, U7 MAX31856, U8 MAX31856, U9 AP63203WU

Commit message: settings ⚙️
Parts:
- C2: moved to F.Cu
- turned C2 to 180 degrees
Changed lines of the file:
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@@
 		)
 	)
+	(footprint "Capacitor_SMD:C_0402_1005Metric"
+		(layer "F.Cu")
+		(at 146.97 95 180)
+		(descr "Capacitor SMD 0402 (1005 Metric), square (rectangular) end terminal, IPC-7351 nominal, (Body size source: IPC-SM-782 page 76, https://www.pcb-3d.com/wordpress/wp-content/uploads/ipc-sm-782a_amendment_1_and_2.pdf), generated with kicad-footprint-generator")
+		(tags "capacitor")
+		(property "Reference" "C2"
+			(at 0 -1.16 0)
+			(layer "F.SilkS")
+			(hide yes)
+			(effects
+				(font
+					(size 1 1)
+					(thickness 0.15)
+				)
+			)
+		)
+		(property "Value" "100nF"
+			(at 0 1.16 0)
+			(layer "F.Fab")
+			(effects
+				(font
+					(size 1 1)
+					(thickness 0.15)
+				)
+			)
+		)
+		(property "Datasheet" "~"
+			(at 0 0 0)
+			(layer "F.Fab")
+			(hide yes)
+			(effects
+				(font
+					(size 1.27 1.27)
+					(thickness 0.15)
+				)
+			)
+		)
+		(property "Description" "Unpolarized capacitor"
+			(at 0 0 0)
+			(layer "F.Fab")
+			(hide yes)
+			(effects
+				(font
+					(size 1.27 1.27)
+					(thickness 0.15)
+				)
+			)
+		)
+		(property ki_fp_filters "C_*")
+		(sheetname "/stm32f1/")
+		(sheetfile "stm32f1.kicad_sch")
+		(attr smd)
+		(fp_line
+			(start -0.107836 0.36)
+			(end 0.107836 0.36)
+			(stroke
+				(width 0.12)
+				(type solid)
+			)
+			(layer "F.SilkS")
+		)
+		(fp_line
+			(start -0.107836 -0.36)
+			(end 0.107836 -0.36)
+			(stroke
+				(width 0.12)
+				(type solid)
+			)
+			(layer "F.SilkS")
+		)
+		(fp_line
+			(start 0.91 0.46)
+			(end -0.91 0.46)
+			(stroke
+				(width 0.05)
+				(type solid)
+			)
+			(layer "F.CrtYd")
+		)
+		(fp_line
+			(start 0.91 -0.46)
+			(end 0.91 0.46)
+			(stroke
+				(width 0.05)
+				(type solid)
+			)
+			(layer "F.CrtYd")
+		)
+		(fp_line
+			(start -0.91 0.46)
+			(end -0.91 -0.46)
+			(stroke
+				(width 0.05)
+				(type solid)
+			)
+			(layer "F.CrtYd")
+		)
+		(fp_line
+			(start -0.91 -0.46)
+			(end 0.91 -0.46)
+			(stroke
+				(width 0.05)
+				(type solid)
+			)
+			(layer "F.CrtYd")
+		)
+		(fp_line
+			(start 0.5 0.25)
+			(end -0.5 0.25)
+			(stroke
+				(width 0.1)
+				(type solid)
+			)
+			(layer "F.Fab")
+		)
+		(fp_line
+			(start 0.5 -0.25)
+			(end 0.5 0.25)
+			(stroke
+				(width 0.1)
+				(type solid)
+			)
+			(layer "F.Fab")
+		)
+		(fp_line
+			(start -0.5 0.25)
+			(end -0.5 -0.25)
+			(stroke
+				(width 0.1)
+				(type solid)
+			)
+			(layer "F.Fab")
+		)
+		(fp_line
+			(start -0.5 -0.25)
+			(end 0.5 -0.25)
+			(stroke
+				(width 0.1)
+				(type solid)
+			)
+			(layer "F.Fab")
+		)
+		(fp_text user "${REFERENCE}"
+			(at 0 0 0)
+			(layer "F.Fab")
+			(effects
+				(font
+					(size 0.25 0.25)
+					(thickness 0.04)
+				)
+			)
+		)
+		(pad "1" smd roundrect
+			(at -0.48 0 180)
+			(size 0.56 0.62)
+			(layers "F.Cu" "F.Mask" "F.Paste")
+			(roundrect_rratio 0.25)
+			(net 9 "+3.3V")
+			(pintype "passive")
+		)
+		(pad "2" smd roundrect
+			(at 0.48 0 180)
+			(size 0.56 0.62)
+			(layers "F.Cu" "F.Mask" "F.Paste")
+			(roundrect_rratio 0.25)
+			(net 5 "GND")
+			(pintype "passive")
+		)
+		(embedded_fonts no)
+		(model "${KICAD9_3DMODEL_DIR}/Capacitor_SMD.3dshapes/C_0402_1005Metric.step"
+			(offset
+				(xyz 0 0 0)
+			)
+			(scale
+				(xyz 1 1 1)
+			)
+			(rotate
+				(xyz 0 0 0)
+			)
+		)
+	)
 	(footprint "Resistor_SMD:R_0402_1005Metric"
 		(layer "F.Cu")
@@
 		(embedded_fonts no)
 	)
-	(footprint "Capacitor_SMD:C_0402_1005Metric"
-		(layer "B.Cu")
-		(at 146.97 95)
-		(descr "Capacitor SMD 0402 (1005 Metric), square (rectangular) end terminal, IPC-7351 nominal, (Body size source: IPC-SM-782 page 76, https://www.pcb-3d.com/wordpress/wp-content/uploads/ipc-sm-782a_amendment_1_and_2.pdf), generated with kicad-footprint-generator")
-		(tags "capacitor")
-		(property "Reference" "C2"
-			(at 0 1.16 0)
-			(layer "B.SilkS")
-			(hide yes)
-			(effects
-				(font
-					(size 1 1)
-					(thickness 0.15)
-				)
-				(justify mirror)
-			)
-		)
-		(property "Value" "100nF"
-			(at 0 -1.16 0)
-			(layer "B.Fab")
-			(effects
-				(font
-					(size 1 1)
-					(thickness 0.15)
-				)
-				(justify mirror)
-			)
-		)
-		(property "Datasheet" "~"
-			(at 0 0 0)
-			(layer "B.Fab")
-			(hide yes)
-			(effects
-				(font
-					(size 1.27 1.27)
-					(thickness 0.15)
-				)
-				(justify mirror)
-			)
-		)
-		(property "Description" "Unpolarized capacitor"
-			(at 0 0 0)
-			(layer "B.Fab")
-			(hide yes)
-			(effects
-				(font
-					(size 1.27 1.27)
-					(thickness 0.15)
-				)
-				(justify mirror)
-			)
-		)
-		(property ki_fp_filters "C_*")
-		(sheetname "/stm32f1/")
-		(sheetfile "stm32f1.kicad_sch")
-		(attr smd)
-		(fp_line
-			(start -0.107836 -0.36)
-			(end 0.107836 -0.36)
-			(stroke
-				(width 0.12)
-				(type solid)
-			)
-			(layer "B.SilkS")
-		)
-		(fp_line
-			(start -0.107836 0.36)
-			(end 0.107836 0.36)
-			(stroke
-				(width 0.12)
-				(type solid)
-			)
-			(layer "B.SilkS")
-		)
-		(fp_line
-			(start -0.91 -0.46)
-			(end -0.91 0.46)
-			(stroke
-				(width 0.05)
-				(type solid)
-			)
-			(layer "B.CrtYd")
-		)
-		(fp_line
-			(start -0.91 0.46)
-			(end 0.91 0.46)
-			(stroke
-				(width 0.05)
-				(type solid)
-			)
-			(layer "B.CrtYd")
-		)
-		(fp_line
-			(start 0.91 -0.46)
-			(end -0.91 -0.46)
-			(stroke
-				(width 0.05)
-				(type solid)
-			)
-			(layer "B.CrtYd")
-		)
-		(fp_line
-			(start 0.91 0.46)
-			(end 0.91 -0.46)
-			(stroke
-				(width 0.05)
-				(type solid)
-			)
-			(layer "B.CrtYd")
-		)
-		(fp_line
-			(start -0.5 -0.25)
-			(end -0.5 0.25)
-			(stroke
-				(width 0.1)
-				(type solid)
-			)
-			(layer "B.Fab")
-		)
-		(fp_line
-			(start -0.5 0.25)
-			(end 0.5 0.25)
-			(stroke
-				(width 0.1)
-				(type solid)
-			)
-			(layer "B.Fab")
-		)
-		(fp_line
-			(start 0.5 -0.25)
-			(end -0.5 -0.25)
-			(stroke
-				(width 0.1)
-				(type solid)
-			)
-			(layer "B.Fab")
-		)
-		(fp_line
-			(start 0.5 0.25)
-			(end 0.5 -0.25)
-			(stroke
-				(width 0.1)
-				(type solid)
-			)
-			(layer "B.Fab")
-		)
-		(fp_text user "${REFERENCE}"
-			(at 0 0 0)
-			(layer "B.Fab")
-			(effects
-				(font
-					(size 0.25 0.25)
-					(thickness 0.04)
-				)
-				(justify mirror)
-			)
-		)
-		(pad "1" smd roundrect
-			(at -0.48 0)
-			(size 0.56 0.62)
-			(layers "B.Cu" "B.Mask" "B.Paste")
-			(roundrect_rratio 0.25)
-			(net 9 "+3.3V")
-			(pintype "passive")
-		)
-		(pad "2" smd roundrect
-			(at 0.48 0)
-			(size 0.56 0.62)
-			(layers "B.Cu" "B.Mask" "B.Paste")
-			(roundrect_rratio 0.25)
-			(net 5 "GND")
-			(pintype "passive")
-		)
-		(embedded_fonts no)
-		(model "${KICAD9_3DMODEL_DIR}/Capacitor_SMD.3dshapes/C_0402_1005Metric.step"
-			(offset
-				(xyz 0 0 0)
-			)
-			(scale
-				(xyz 1 1 1)
-			)
-			(rotate
-				(xyz 0 0 0)
-			)
-		)
-	)
 	(footprint "Images:NDXP-Logo"
 		(layer "B.Cu")
@@
 		(polygon
 			(pts
-				(xy 108.6 46.7) (xy 110.9 148.1) (xy 186.2 149.1) (xy 185.1 48.1)
+				(xy 109.9 46.8) (xy 112.2 148.2) (xy 187.5 149.2) (xy 186.4 48.2)
 			)
 		)

Commit message: Moved Mary to avoid MCU
Parts:
- moved G*** 9.82 mm to (149.8, 111.8)

Commit message: ROuted 5V Power
Parts:
- removed the C48 at (124.2, 118.6)
- removed the U12 at (127.6, 120.0)
Routing:
- net +5V: track 0.00 -> 276.3 mm

Commit message: routed initial🛣️
Parts:
- moved R33 3.36 mm to (139.7, 102.9)
- moved C1 1.69 mm to (144.6, 107.9), turned to -135 degrees
- moved R31 1.50 mm to (134.8, 106.5)
- moved U13 1.49 mm to (137.4, 103.9)
- moved C7 1.25 mm to (142.5, 105.8)
- moved C8 1.20 mm to (134.8, 104.1)
- moved R1 1.05 mm to (140.5, 100.6), turned to 135 degrees
- moved R32 1.00 mm to (163.1, 105.6)
- moved C9 0.70 mm to (163.1, 103.2)
- moved C5 0.62 mm to (142.1, 98.5)
- moved R3 0.62 mm to (144.5, 96.3)
- moved R23 0.44 mm to (143.9, 107.2), turned to -135 degrees
- moved R22 0.41 mm to (139.7, 104.8)
Routing:
- net +5V: track 276.3 -> 174.8 mm, vias 0 -> 1
- net /stm32f1/SPI1_SCK: track 0.00 -> 35.4 mm
- net CH_08: track 0.00 -> 27.8 mm
- net CH_07: track 0.00 -> 27.4 mm
- net CH_02: track 0.00 -> 21.3 mm
- net CH_13: track 0.00 -> 20.5 mm
- net CH_09: track 0.00 -> 19.3 mm
- net CH_06: track 0.00 -> 18.9 mm
- net SDA_5V: track 0.00 -> 13.9 mm
- net SCL_5V: track 0.00 -> 13.2 mm
- net CH_03: track 0.00 -> 12.9 mm
- net CH_12: track 0.00 -> 12.0 mm
- net CH_10: track 0.00 -> 10.9 mm
- net CH_05: track 0.00 -> 10.5 mm
- net CH_04: track 0.00 -> 7.39 mm
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- added copper zone on In2.Cu, net +3.3V
- added copper zone on In1.Cu, net GND
Other:
- copper layers 2 -> 4

Commit message: 3.3 partially routed, to avoid signal
Parts:
- moved C29 4.63 mm to (173.0, 100.8)
- moved C17 0.92 mm to (124.6, 98.1)
Routing:
- net +3.3V: track 0.00 -> 42.8 mm, vias 0 -> 29
- net +5V: track 174.8 -> 202.8 mm, vias 1 -> 5
- net GND: track 0.00 -> 2.26 mm, vias 0 -> 1
- net /Hardware_Safe/BW1: track 0.00 -> 1.20 mm, vias 0 -> 1

Commit message: signal
Parts:
- moved J21 13.2 mm to (159.6, 65.9)
- moved R11 11.4 mm to (153.7, 89.2), turned to -135 degrees
- moved C20 11.2 mm to (152.3, 90.6), turned to -135 degrees
- moved C10 10.1 mm to (143.4, 91.2), turned to 135 degrees
- moved C15 10.0 mm to (124.5, 95.8), turned to 90 degrees
- moved C22 9.94 mm to (154.9, 89.5), turned to -135 degrees
- moved C25 9.87 mm to (173.0, 95.7), turned to -90 degrees
- moved C19 9.84 mm to (133.3, 99.9), turned to 0 degrees
- moved C23 9.82 mm to (173.0, 97.5), turned to 90 degrees
- moved C50 9.81 mm to (165.9, 91.3), turned to 180 degrees
- moved R10 9.80 mm to (152.2, 92.2), turned to 45 degrees
- moved R6 9.57 mm to (140.6, 89.9), turned to -45 degrees
- moved C24 9.11 mm to (153.6, 90.8), turned to 45 degrees
- moved R8 8.85 mm to (125.5, 98.5), turned to 90 degrees
- moved C12 8.81 mm to (143.8, 94.5), turned to 45 degrees
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Routing:
- net /Accelerometer/ACC_SCL: track 0.00 -> 53.0 mm, vias 0 -> 2
- net /stm32f1/SPI1_MISO: track 0.00 -> 51.9 mm, vias 0 -> 3
- net /Accelerometer/ACC_SDA: track 0.00 -> 50.6 mm, vias 0 -> 2
- net /stm32f1/SPI1_MOSI: track 0.00 -> 50.3 mm, vias 0 -> 3
- net Net-(J21-Pin_1): track 0.00 -> 46.6 mm, vias 0 -> 1
- net Net-(J21-Pin_2): track 0.00 -> 44.6 mm, vias 0 -> 1
- net Net-(J19-Pin_2): track 0.00 -> 39.2 mm, vias 0 -> 1
- net Net-(J19-Pin_1): track 0.00 -> 38.5 mm, vias 0 -> 1
- net Net-(J18-Pin_1): track 0.00 -> 35.0 mm, vias 0 -> 1
- net Net-(J20-Pin_1): track 0.00 -> 31.5 mm, vias 0 -> 1
- net +3.3V: track 42.8 -> 14.9 mm, vias 29 -> 0
- net Net-(J20-Pin_2): track 0.00 -> 27.7 mm, vias 0 -> 1
- net Net-(J18-Pin_2): track 0.00 -> 25.7 mm, vias 0 -> 1
- net /stm32f1/TC1_CS: track 0.00 -> 25.5 mm, vias 0 -> 2
- net SW_PWR: track 0.00 -> 23.5 mm
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
Commit message: newest
Routing:
- net +3.3V: track 14.9 -> 8.56 mm
- net GND: track 0.00 -> 3.82 mm, vias 0 -> 1
- net +5V: track 202.7 -> 199.3 mm, vias 5 -> 3
- net Net-(C48-Pad1): track 0.00 -> 2.08 mm
- net /stm32f1/SPI1_MISO: track 51.9 -> 53.4 mm
- net Net-(C48-Pad2): track 0.00 -> 0.98 mm, vias 0 -> 1
- net Net-(U7-T-): track 0.00 -> 0.63 mm
- net /RS-485/TX_RS485: track 0.00 -> 0.52 mm

Commit message: Routed some stuff
Parts:
- moved TP1 3.35 mm to (151.7, 94.4)
- moved C21 2.28 mm to (172.1, 100.6)
- moved R13 2.28 mm to (172.1, 98.7)
- moved R12 2.28 mm to (172.1, 96.8)
- moved C23 2.28 mm to (173.1, 99.8)
- moved C29 1.83 mm to (173.1, 98.0)
- moved R2 0.40 mm to (149.3, 94.8), turned to -90 degrees
- moved C25 0.38 mm to (173.1, 96.1)
- moved C2 0.30 mm to (147.2, 94.8), turned to -90 degrees
Routing:
- net SCL_5V: track 13.2 -> 92.2 mm
- net /Solenoids/S1: track 0.00 -> 50.2 mm, vias 0 -> 4
- net Net-(J30-Pin_3): track 0.00 -> 46.7 mm
- net /Solenoids/S2: track 0.00 -> 41.5 mm, vias 0 -> 6
- net /Solenoids/S4: track 0.00 -> 41.1 mm, vias 0 -> 2
- net Net-(J30-Pin_2): track 0.00 -> 37.2 mm
- net en: track 0.00 -> 36.0 mm, vias 0 -> 2
- net /RS-485/RX_RS485: track 0.00 -> 34.5 mm, vias 0 -> 2
- net /Pyro/PYRO1: track 0.00 -> 34.0 mm, vias 0 -> 2
- net /Solenoids/S3: track 0.00 -> 32.7 mm, vias 0 -> 2
- net /RS-485/TX_RS485: track 0.52 -> 29.0 mm, vias 0 -> 2
- net /Hardware_Safe/K1: track 2.95 -> 30.7 mm
- net FB: track 0.00 -> 27.6 mm, vias 0 -> 2
- net Net-(C31-Pad1): track 0.00 -> 24.8 mm, vias 0 -> 2
- net /ADS1231/LC_DRDY/DOUT: track 0.00 -> 21.9 mm, vias 0 -> 2
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