File: stm32f1.kicad_sch (KiCad schematic)
At the start: 11 parts, among them SW1 SW_Push, SW2 SW_Push, U2 STM32F103C8Tx

Commit message: adcs
Parts:
- added R4, R5: 4.7K, symbol Device:R
Connections:
- net +3.3V: now also R4.1, R5.1
- net SCL: now reaches U2.42 (PB6)
- net SCL: now also R5.2
- net SDA: now reaches U2.43 (PB7)
- net SDA: now also R4.2
Other:
- note added: "I2C Pullup"

Commit message: power
Connections:
- net SPI1_SCK: now reaches U2.15 (PA5)
- net SPI1_MISO: now reaches U2.16 (PA6)
- net SPI1_MOSI: now reaches U2.17 (PA7)
Changed lines of the file:
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@@
+		)
+	)
+	(hierarchical_label "SPI1_MOSI"
+		(shape input)
+		(at 158.75 88.9 0)
+		(effects
+			(font
+				(size 1.27 1.27)
+			)
+			(justify left)
+		)
+	)
+	(hierarchical_label "SPI1_SCK"
+		(shape input)
+		(at 158.75 83.82 0)
+		(effects
+			(font
+				(size 1.27 1.27)
+			)
+			(justify left)
 		)
 	)
@@
 		(effects
 			(font
+				(size 1.27 1.27)
+			)
+			(justify left)
+		)
+	)
+	(hierarchical_label "SPI1_MISO"
+		(shape input)
+		(at 158.75 86.36 0)
+		(effects
+			(font

Commit message: reg🟡
Parts:
- renumbered C6 to C2, C7 to C3, C9 to C4, C10 to C5, C11 to C6, C12 to C7, R5 to R1, R4 to R2, R1 to R3, SW2 to SW1, SW1 to SW2, U2 to U1
Connections:
- net TC3_CS: now reaches U1.13 (PA3)
- net TC4_CS: now reaches U1.14 (PA4)
- net TC1_CS: now reaches U1.18 (PB0)
- net TC2_CS: now reaches U1.19 (PB1)

Commit message: layout🏄‍♂️
Parts:
- removed C1: 100nF, symbol Device:C
- added C33: 100nF, Capacitor_SMD:C_0402_1005Metric, symbol Device:C
- C2, C3, C4, C6: footprint (none) -> Capacitor_SMD:C_0402_1005Metric
- C5: footprint (none) -> Capacitor_SMD:C_0805_2012Metric
- C7: footprint (none) -> Capacitor_SMD:C_0603_1608Metric
- R1, R2: footprint (none) -> Resistor_SMD:R_0402_1005Metric
- R3: footprint (none) -> Resistor_SMD:R_0603_1608Metric
Connections:
- net GND: now also C33.2
- net at SW1.2, U1.7 (NRST): now also C33.1

Commit message: plug🔌
Connections:
- net TC3_CS: now also U1.11 (PA1); no longer U1.13 (PA3)
- net TC4_CS: now also U1.10 (PA0); no longer U1.14 (PA4)
- net UART_2_TX: now reaches U1.12 (PA2)
- net I2C2_SDA: now reaches U1.21 (PB10)
- net I2C2_SCL: now reaches U1.22 (PB11)
- net SCL renamed I2C1_SCL
- net SDA renamed I2C1_SDA
- new net DIR_RS485: U1.14 (PA4)
- new net UART_2_RX: U1.13 (PA3)
Changed lines of the file:
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@@
+		)
+	)
+	(hierarchical_label "I2C2_SCL"
+		(shape input)
+		(at 123.19 127 180)
+		(effects
+			(font
+				(size 1.27 1.27)
+			)
+			(justify right)
+		)
+	)
+	(hierarchical_label "UART_2_RX"
+		(shape input)
+		(at 158.75 78.74 0)
+		(effects
+			(font
+				(size 1.27 1.27)
+			)
+			(justify left)
 		)
 	)
@@
 		)
 	)
-	(hierarchical_label "TC3_CS"
+	(hierarchical_label "DIR_RS485"
 		(shape input)
-		(at 158.75 78.74 0)
+		(at 158.75 81.28 0)
 		(effects
 			(font
@@
 		)
 	)
-	(hierarchical_label "SCL"
+	(hierarchical_label "TC3_CS"
+		(shape input)
+		(at 158.75 73.66 0)
+		(effects
+			(font
+				(size 1.27 1.27)
+			)
+			(justify left)
+		)
+	)
+	(hierarchical_label "I2C2_SDA"
+		(shape input)
+		(at 123.19 124.46 180)
+		(effects
+			(font
+				(size 1.27 1.27)
+			)
+			(justify right)
+		)
+	)
+	(hierarchical_label "I2C1_SCL"
 		(shape input)
 		(at 91.44 114.3 180)
@@
 	(hierarchical_label "TC4_CS"
 		(shape input)
-		(at 158.75 81.28 0)
+		(at 158.75 71.12 0)
+		(effects
+			(font
+				(size 1.27 1.27)
+			)
+			(justify left)
+		)
+	)
+	(hierarchical_label "UART_2_TX"
+		(shape input)
+		(at 158.75 76.2 0)
 		(effects
 			(font
@@
 		)
 	)
-	(hierarchical_label "SDA"
+	(hierarchical_label "I2C1_SDA"
 		(shape input)
 		(at 91.44 116.84 180)

Commit message: Connected solenoids, some error fixes
Connections:
- net S1: now reaches U1.25 (PB12)
- net S2: now reaches U1.26 (PB13)
- net S3: now reaches U1.27 (PB14)
- net S4: now reaches U1.28 (PB15)
Changed lines of the file:
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@@
+	)
+	(junction
+		(at 115.57 72.39)
+		(diameter 0)
+		(color 0 0 0 0)
 	)
 	(junction
@@
 	(wire
 		(pts
-			(xy 109.22 72.39) (xy 123.19 72.39)
+			(xy 109.22 72.39) (xy 115.57 72.39)
 		)
 		(stroke
@@
 	(wire
 		(pts
+			(xy 115.57 72.39) (xy 123.19 72.39)
+		)
+		(stroke
+			(width 0)
+			(type default)
+		)
+	)
+	(wire
+		(pts
 			(xy 224.79 54.61) (xy 234.95 54.61)
 		)
@@
 		)
 	)
+	(hierarchical_label "S1"
+		(shape input)
+		(at 123.19 129.54 180)
+		(effects
+			(font
+				(size 1.27 1.27)
+			)
+			(justify right)
+		)
+	)
 	(hierarchical_label "TC3_CS"
 		(shape input)
@@
 		)
 	)
+	(hierarchical_label "S2"
+		(shape input)
+		(at 123.19 132.08 180)
+		(effects
+			(font
+				(size 1.27 1.27)
+			)
+			(justify right)
+		)
+	)
 	(hierarchical_label "TC1_CS"
 		(shape input)
@@
 		)
 	)
+	(hierarchical_label "S3"
+		(shape input)
+		(at 123.19 134.62 180)
+		(effects
+			(font
+				(size 1.27 1.27)
+			)
+			(justify right)
+		)
+	)
 	(hierarchical_label "TC2_CS"
 		(shape input)
 		(at 123.19 101.6 180)
+		(effects
+			(font
+				(size 1.27 1.27)
+			)
+			(justify right)
+		)
+	)
+	(hierarchical_label "S4"
+		(shape input)
+		(at 123.19 137.16 180)
 		(effects
 			(font
@@
 					(unit 1)
 				)
+			)
+		)
+	)
+	(symbol
+		(lib_id "power:PWR_FLAG")
+		(at 115.57 72.39 0)
+		(unit 1)
+		(exclude_from_sim no)
+		(in_bom yes)
+		(on_board yes)
+		(dnp no)
+		(fields_autoplaced yes)
+		(property "Reference" "#FLG03"
+			(at 115.57 70.485 0)
+			(effects
+				(font
+					(size 1.27 1.27)
+				)
+				(hide yes)
+			)
+		)
+		(property "Value" "PWR_FLAG"
+			(at 115.57 67.31 0)
+			(effects
+				(font
+					(size 1.27 1.27)
+				)
+			)
+		)
+		(property "Footprint" ""
+			(at 115.57 72.39 0)
+			(effects
+				(font
+					(size 1.27 1.27)
+				)
+				(hide yes)
+			)
+		)
+		(property "Datasheet" "~"
+			(at 115.57 72.39 0)
+			(effects
+				(font
+					(size 1.27 1.27)
+				)
+				(hide yes)
+			)
+		)
+		(property "Description" "Special symbol for telling ERC where power comes from"
+			(at 115.57 72.39 0)
+			(effects
+				(font
+					(size 1.27 1.27)
+				)
+				(hide yes)
+			)
+		)
+		(pin "1"
+		)
+		(instances
+			(project ""
+				(path "/bb73515c-a1ce-4448-8899-3a433fb04c26/9cbbe99d-ef26-4275-9460-efaf874d2391"
+					(reference "#FLG03")
+					(unit 1)
+				)

Commit message: arranged board
Connections:
- net BW1: now reaches U1.20 (PB2)
- net PYRO1: now reaches U1.29 (PA8)
- net K1: now reaches U1.5 (PD0)
- net K2: now reaches U1.6 (PD1)
Changed lines of the file:
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@@
+		)
+	)
+	(hierarchical_label "PYRO1"
+		(shape input)
+		(at 158.75 91.44 0)
+		(effects
+			(font
+				(size 1.27 1.27)
+			)
+			(justify left)
+		)
+	)
+	(hierarchical_label "K1"
+		(shape input)
+		(at 123.19 81.28 180)
+		(effects
+			(font
+				(size 1.27 1.27)
+			)
+			(justify right)
 		)
 	)
@@
 		)
 	)
+	(hierarchical_label "BW1"
+		(shape input)
+		(at 123.19 104.14 180)
+		(effects
+			(font
+				(size 1.27 1.27)
+			)
+			(justify right)
+		)
+	)
 	(hierarchical_label "TC1_CS"
 		(shape input)
@@
 		(shape input)
 		(at 123.19 137.16 180)
+		(effects
+			(font
+				(size 1.27 1.27)
+			)
+			(justify right)
+		)
+	)
+	(hierarchical_label "K2"
+		(shape input)
+		(at 123.19 83.82 180)
 		(effects
 			(font
@@
 		(dnp no)
 		(property "Reference" "C33"
-			(at 114.3 78.74 0)
+			(at 109.728 82.55 0)
 			(effects
 				(font
@@
 		)
 		(property "Value" "100nF"
-			(at 114.3 81.28 0)
-			(effects
-				(font
+			(at 109.728 85.09 0)
+			(effects
+				(font

Commit message: added leds🔴🟡🔵
Parts:
- added D10: Yellow, LED_SMD:LED_0603_1608Metric, symbol Device:LED
- added D11: Blue, LED_SMD:LED_0603_1608Metric, symbol Device:LED
- added D9: Red, LED_SMD:LED_0603_1608Metric, symbol Device:LED
- added R28, R29, R30: 100, Resistor_SMD:R_0402_1005Metric, symbol Device:R
- renumbered C33 to C1
Connections:
- net +3.3V: now also R28.1, R29.1, R30.1
- net at U1.2 (PC13): now also D9.1 (K)
- net at U1.3 (PC14): now also D10.1 (K)
- net at U1.4 (PC15): now also D11.1 (K)
- new net: D11.2 (A), R30.2
- new net: D10.2 (A), R29.2
- new net: D9.2 (A), R28.2
Other:
- moved on the sheet: C1, SW1
