File: stm32f1.kicad_sch (KiCad schematic)
At the start: 19 parts, among them SW1 SW_Push, SW2 SW_Push, U1 STM32F103C8Tx

Commit message: bomupdate
Parts:
- D10: JLC# C965808 -> C19273150
- D11: JLC# C965807 -> C19171394
- D9: JLC# C965799 -> C19171390
- R28, R29, R30: value 100 -> 100Ω
Changed lines of the file:
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@@
 			)
 		)
-		(property "Value" "100"
+		(property "Value" "100Ω"
 			(at 109.728 93.98 90)
 			(effects
@@
 			)
 		)
-		(property "JLC#" "C965807"
+		(property "JLC#" "C19171394"
 			(at 115.57 93.98 0)
 			(effects
@@
 			)
 		)
-		(property "Value" "100"
+		(property "Value" "100Ω"
 			(at 109.728 91.44 90)
 			(effects
@@
 			)
 		)
-		(property "JLC#" "C965799"
+		(property "JLC#" "C19171390"
 			(at 114.808 86.36 0)
 			(effects
@@
 			)
 		)
-		(property "JLC#" "C965808"
+		(property "JLC#" "C19273150"
 			(at 114.554 90.424 0)
 			(effects
@@
 			)
 		)
-		(property "Value" "100"
+		(property "Value" "100Ω"
 			(at 109.728 88.9 90)
 			(effects
