File: ADCs.kicad_sch (KiCad schematic)
At the start: 4 parts, among them U3 ADS7828, U4 ADS7828

Commit message: added luke name
Parts:
- added U5: MAX31855KASA, Package_SO:SOIC-8_3.9x4.9mm_P1.27mm, symbol Sensor_Temperature:MAX31855KASA
Changed lines of the file:
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@@
+	)
+	(symbol
+		(lib_id "Sensor_Temperature:MAX31855KASA")
+		(at 185.42 48.26 0)
+		(unit 1)
+		(exclude_from_sim no)
+		(in_bom yes)
+		(on_board yes)
+		(dnp no)
+		(fields_autoplaced yes)
+		(property "Reference" "U5"
+			(at 187.5633 35.56 0)
+			(effects
+				(font
+					(size 1.27 1.27)
+				)
+				(justify left)
+			)
+		)
+		(property "Value" "MAX31855KASA"
+			(at 187.5633 38.1 0)
+			(effects
+				(font
+					(size 1.27 1.27)
+				)
+				(justify left)
+			)
+		)
+		(property "Footprint" "Package_SO:SOIC-8_3.9x4.9mm_P1.27mm"
+			(at 187.96 58.42 0)
+			(effects
+				(font
+					(size 1.27 1.27)
+					(italic yes)
+				)
+				(justify left)
+				(hide yes)
+			)
+		)
+		(property "Datasheet" "http://datasheets.maximintegrated.com/en/ds/MAX31855.pdf"
+			(at 187.96 60.96 0)
+			(effects
+				(font
+					(size 1.27 1.27)
+				)
+				(justify left)
+				(hide yes)
+			)
+		)
+		(property "Description" "Cold Junction K-type Thermocouple Interface, SPI, SOIC-8"
+			(at 187.96 55.88 0)
+			(effects
+				(font
+					(size 1.27 1.27)
+				)
+				(justify left)
+				(hide yes)
+			)
+		)
+		(pin "6"
+		)
+		(pin "4"
+		)
+		(pin "7"
+		)
+		(pin "2"
+		)
+		(pin "1"
+		)
+		(pin "5"
+		)
+		(pin "3"
+		)
+		(pin "8"
+		)
+		(instances
+			(project ""
+				(path "/bb73515c-a1ce-4448-8899-3a433fb04c26/c5809e31-49fa-4035-9e50-9a02f65a2597"
+					(reference "U5")
+					(unit 1)
+				)
+			)
+		)
 	)
 	(symbol

Commit message: power
Parts:
- removed U5: MAX31855KASA, Package_SO:SOIC-8_3.9x4.9mm_P1.27mm, symbol Sensor_Temperature:MAX31855KASA
Other:
- moved on the sheet: C2, C3, U3, U4

Commit message: reg🟡
Parts:
- renumbered C2 to C8, C3 to C9

Commit message: layout🏄‍♂️
Parts:
- added J10, J11, J12, J13, J14, J15, J16, J17, J18, J19, J4, J5, J6, J7, J8, J9: Conn_01x03, TerminalBlock_Phoenix:TerminalBlock_Phoenix_MPT-0,5-3-2.54_1x03_P2.54mm_Horizontal, symbol Connector_Generic:Conn_01x03
- C8, C9: footprint (none) -> Capacitor_SMD:C_0603_1608Metric
Connections:
- net +5V: now also J10.1 (Pin_1), J11.1 (Pin_1), J12.1 (Pin_1), J13.1 (Pin_1), J14.1 (Pin_1), J15.1 (Pin_1), J16.1 (Pin_1), J17.1 (Pin_1), J18.1 (Pin_1), J19.1 (Pin_1), J4.1 (Pin_1), J5.1 (Pin_1), J6.1 (Pin_1), J7.1 (Pin_1), J8.1 (Pin_1), J9.1 (Pin_1)
- net CH_00: now also J4.2 (Pin_2)
- net CH_01: now also J5.2 (Pin_2)
- net CH_02: now also J8.2 (Pin_2)
- net CH_03: now also J10.2 (Pin_2)
- net CH_04: now also J6.2 (Pin_2)
- net CH_05: now also J7.2 (Pin_2)
- net CH_06: now also J9.2 (Pin_2)
- net CH_07: now also J11.2 (Pin_2)
- net CH_08: now also J12.2 (Pin_2)
- net CH_09: now also J14.2 (Pin_2)
- net CH_10: now also J16.2 (Pin_2)
- net CH_11: now also J18.2 (Pin_2)
- net CH_12: now also J13.2 (Pin_2)
- net CH_13: now also J15.2 (Pin_2)
- net CH_14: now also J17.2 (Pin_2)
- net CH_15: now also J19.2 (Pin_2)
- net GND: now also J10.3 (Pin_3), J11.3 (Pin_3), J12.3 (Pin_3), J13.3 (Pin_3), J14.3 (Pin_3), J15.3 (Pin_3), J16.3 (Pin_3), J17.3 (Pin_3), J18.3 (Pin_3), J19.3 (Pin_3), J4.3 (Pin_3), J5.3 (Pin_3), J6.3 (Pin_3), J7.3 (Pin_3), J8.3 (Pin_3), J9.3 (Pin_3)
Other:
- note added: "Terminal Blocks"
- moved on the sheet: C8, C9, U3, U4

Commit message: Fixed Filters on ADCs
Connections:
- net +3.3V: no longer C8.2, C9.2
- net GND: now also C8.2, C9.2
Other:
- moved on the sheet: C8, C9
Changed lines of the file:
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@@
 	)
 	(junction
-		(at 76.2 74.93)
-		(diameter 0)
-		(color 0 0 0 0)
-	)
-	(junction
 		(at 125.73 116.84)
 		(diameter 0)
@@
 	)
 	(junction
-		(at 125.73 76.2)
-		(diameter 0)
-		(color 0 0 0 0)
-	)
-	(junction
 		(at 86.36 106.68)
 		(diameter 0)
@@
 	(wire
 		(pts
-			(xy 125.73 76.2) (xy 125.73 77.47)
+			(xy 125.73 68.58) (xy 125.73 77.47)
 		)
 		(stroke
@@
 	(wire
 		(pts
-			(xy 76.2 74.93) (xy 76.2 76.2)
-		)
-		(stroke
-			(width 0)
-			(type default)
-		)
-	)
-	(wire
-		(pts
 			(xy 234.95 72.39) (xy 236.22 72.39)
 		)
@@
 	(wire
 		(pts
-			(xy 76.2 67.31) (xy 83.82 67.31)
+			(xy 76.2 67.31) (xy 87.63 67.31)
 		)
 		(stroke
@@
 	(wire
 		(pts
-			(xy 125.73 76.2) (xy 133.35 76.2)
-		)
-		(stroke
-			(width 0)
-			(type default)
-		)
-	)
-	(wire
-		(pts
 			(xy 115.57 107.95) (xy 115.57 116.84)
 		)
@@
 	(wire
 		(pts
-			(xy 125.73 68.58) (xy 125.73 76.2)
+			(xy 194.31 67.31) (xy 195.58 67.31)
 		)
 		(stroke
@@
 	(wire
 		(pts
-			(xy 194.31 67.31) (xy 195.58 67.31)
+			(xy 173.99 132.08) (xy 175.26 132.08)
 		)
 		(stroke
@@
 	(wire
 		(pts
-			(xy 173.99 132.08) (xy 175.26 132.08)
+			(xy 87.63 74.93) (xy 87.63 76.2)
 		)
 		(stroke
@@
 	(wire
 		(pts
-			(xy 76.2 74.93) (xy 83.82 74.93)
-		)
-		(stroke
-			(width 0)
-			(type default)
-		)
-	)
-	(wire
-		(pts
 			(xy 234.95 137.16) (xy 236.22 137.16)
 		)
@@
 	(wire
 		(pts
-			(xy 76.2 67.31) (xy 76.2 74.93)
+			(xy 76.2 67.31) (xy 76.2 76.2)
 		)
 		(stroke
@@
 	(wire
 		(pts
-			(xy 125.73 68.58) (xy 133.35 68.58)
+			(xy 125.73 68.58) (xy 135.89 68.58)
 		)
 		(stroke
@@
 	)
 	(symbol
+		(lib_id "power:GND")
+		(at 87.63 76.2 0)
+		(unit 1)
+		(exclude_from_sim no)
+		(in_bom yes)
+		(on_board yes)
+		(dnp no)
+		(fields_autoplaced yes)
+		(property "Reference" "#PWR090"
+			(at 87.63 82.55 0)
+			(effects
+				(font
+					(size 1.27 1.27)
+				)
+				(hide yes)
+			)
+		)
+		(property "Value" "GND"
+			(at 87.63 81.28 0)
+			(effects
+				(font
+					(size 1.27 1.27)
+				)
+			)
+		)
+		(property "Footprint" ""
+			(at 87.63 76.2 0)
+			(effects
+				(font
+					(size 1.27 1.27)
+				)
+				(hide yes)
+			)
+		)
+		(property "Datasheet" ""
+			(at 87.63 76.2 0)
+			(effects
+				(font
+					(size 1.27 1.27)
+				)
+				(hide yes)
+			)
+		)
+		(property "Description" "Power symbol creates a global label with name \"GND\" , ground"
+			(at 87.63 76.2 0)
+			(effects
+				(font
+					(size 1.27 1.27)
+				)
+				(hide yes)
+			)
+		)
+		(pin "1"
+		)
+		(instances
+			(project "Alpha_Breakout"
+				(path "/bb73515c-a1ce-4448-8899-3a433fb04c26/c5809e31-49fa-4035-9e50-9a02f65a2597"
+					(reference "#PWR090")
+					(unit 1)
+				)
+			)
+		)
+	)
+	(symbol
 		(lib_id "power:+5V")
 		(at 194.31 87.63 0)
@@
 	(symbol
 		(lib_id "Device:C")
-		(at 83.82 71.12 0)
+		(at 87.63 71.12 0)
 		(unit 1)
 		(exclude_from_sim no)
@@
 		(fields_autoplaced yes)
 		(property "Reference" "C8"
-			(at 87.63 69.8499 0)
+			(at 91.44 69.8499 0)
 			(effects
 				(font
@@
 		)
 		(property "Value" "1uF"
-			(at 87.63 72.3899 0)
+			(at 91.44 72.3899 0)
 			(effects
 				(font
@@
 		)
 		(property "Footprint" "Capacitor_SMD:C_0603_1608Metric"
-			(at 84.7852 74.93 0)
+			(at 88.5952 74.93 0)
 			(effects
 				(font
@@
 		)
 		(property "Datasheet" "~"
-			(at 83.82 71.12 0)
+			(at 87.63 71.12 0)
 			(effects
 				(font
@@
 		)
 		(property "Description" "Unpolarized capacitor"
-			(at 83.82 71.12 0)
+			(at 87.63 71.12 0)
 			(effects
 				(font
@@
 	(symbol
 		(lib_id "Device:C")
-		(at 133.35 72.39 0)
+		(at 135.89 72.39 0)
 		(unit 1)
 		(exclude_from_sim no)
@@
 		(fields_autoplaced yes)
 		(property "Reference" "C9"
-			(at 137.16 71.1199 0)
+			(at 139.7 71.1199 0)
 			(effects
 				(font
@@
 		)
 		(property "Value" "1uF"
-			(at 137.16 73.6599 0)
+			(at 139.7 73.6599 0)
 			(effects
 				(font
@@
 		)
 		(property "Footprint" "Capacitor_SMD:C_0603_1608Metric"
-			(at 134.3152 76.2 0)
+			(at 136.8552 76.2 0)
 			(effects
 				(font
@@
 		)
 		(property "Datasheet" "~"
-			(at 133.35 72.39 0)
+			(at 135.89 72.39 0)
 			(effects
 				(font
@@
 		)
 		(property "Description" "Unpolarized capacitor"
-			(at 133.35 72.39 0)
+			(at 135.89 72.39 0)
 			(effects
 				(font
@@
 					(unit 1)
 				)
+			)
+		)
+	)
+	(symbol
+		(lib_id "power:GND")
+		(at 135.89 76.2 0)
+		(unit 1)
+		(exclude_from_sim no)
+		(in_bom yes)
+		(on_board yes)
+		(dnp no)
+		(fields_autoplaced yes)
+		(property "Reference" "#PWR091"
+			(at 135.89 82.55 0)
+			(effects
+				(font
+					(size 1.27 1.27)
+				)
+				(hide yes)
+			)
+		)
+		(property "Value" "GND"
+			(at 135.89 81.28 0)
+			(effects
+				(font
+					(size 1.27 1.27)
+				)
+			)
+		)
+		(property "Footprint" ""
+			(at 135.89 76.2 0)
+			(effects
+				(font
+					(size 1.27 1.27)
+				)
+				(hide yes)
+			)
+		)
+		(property "Datasheet" ""
+			(at 135.89 76.2 0)
+			(effects
+				(font
+					(size 1.27 1.27)
+				)
+				(hide yes)
+			)
+		)
+		(property "Description" "Power symbol creates a global label with name \"GND\" , ground"
+			(at 135.89 76.2 0)
+			(effects
+				(font
+					(size 1.27 1.27)
+				)
+				(hide yes)
+			)
+		)
+		(pin "1"
+		)
+		(instances
+			(project "Alpha_Breakout"
+				(path "/bb73515c-a1ce-4448-8899-3a433fb04c26/c5809e31-49fa-4035-9e50-9a02f65a2597"
+					(reference "#PWR091")
+					(unit 1)
+				)

Commit message: Not Entirely Sure
Parts:
- added TP3, TP4: TestPoint, TestPoint:TestPoint_Pad_D1.5mm, symbol Connector:TestPoint
Connections:
- net +5V: now also TP3.1, TP4.1

Commit message: added leds🔴🟡🔵
Parts:
- renumbered J8 to J10, J9 to J11, J16 to J12, J17 to J13, J10 to J14, J11 to J15, J18 to J16, J19 to J17, J4 to J2, J6 to J3, J12 to J4, J13 to J5, J5 to J6, J14 to J8, J15 to J9, TP3 to TP2, TP4 to TP3

Commit message: lots🅿️
Parts:
- added R22, R33: 4.7K, Resistor_SMD:R_0402_1005Metric, symbol Device:R
- added R31, R32: 5, symbol Device:R
- added U13: TCA9517ADGK, Package_SO:VSSOP-8_3x3mm_P0.65mm, symbol Logic_LevelTranslator:TCA9517ADGK
Connections:
- net +3.3V: now also U13.1 (VCCA); no longer C8.1, C9.1, U3.16 (VDD), U4.12 (A0), U4.16 (VDD)
- net +5V: now also U4.12 (A0), R22.1, R31.1, R32.1, R33.1, U13.8 (VCCB)
- net GND: now also U13.4 (GND)
- net SCL: now also U13.2 (SCLA); no longer U3.14 (SCL), U4.14 (SCL)
- net SDA: now also U13.3 (SDAA); no longer U3.15 (SDA), U4.15 (SDA)
- new net: C9.1, R32.2, U4.16 (VDD)
- new net: C8.1, R31.2, U3.16 (VDD)
- new net SCL_5V: R22.2, U13.7 (SCLB), U3.14 (SCL), U4.14 (SCL)
- new net SDA_5V: R33.2, U13.6 (SDAB), U3.15 (SDA), U4.15 (SDA)
- no-connect marks 0 -> 1
Other:
- note added: "Level Shifter"
- note added: "internal pullup to VCCB"
- moved on the sheet: C9, TP3, U4
