File: Solenoids.kicad_sch (KiCad schematic)
At the start: 2 parts, among them Q1 CSD13381F4

Commit message: oops I forgot to specify resistor footprint
Parts:
- added D1, D2, D3, D4: D, Diode_SMD:D_SOD-123, symbol Device:D
- added J25, J26, J27, J28: Conn_01x02, TerminalBlock_Phoenix:TerminalBlock_Phoenix_MPT-0,5-2-2.54_1x02_P2.54mm_Horizontal, symbol Connector_Generic:Conn_01x02
- added Q2, Q3, Q4: CSD13381F4, CSD13381F4:DFN100X60X35-3N, symbol CSD13381F4:CSD13381F4
- added R19, R21, R23, R25: 100k, Resistor_SMD:R_0603_1608Metric, symbol Device:R
- added R20, R22, R24: 160, Resistor_SMD:R_0603_1608Metric, symbol Device:R
- R18: value R -> 160; footprint (none) -> Resistor_SMD:R_0603_1608Metric
Connections:
- net GND: now also Q2.2, Q3.2, Q4.2, R19.2, R21.2, R23.2, R25.2
- net at Q1.1, R18.2: now also R19.1
- net at Q1.3: now also D1.2 (A), J25.2 (Pin_2)
- new net: D2.2 (A), J26.2 (Pin_2), Q2.3
- new net: Q2.1, R20.2, R21.1
- new net: D3.2 (A), J27.2 (Pin_2), Q3.3
- new net: Q4.1, R24.2, R25.1
- new net: D4.2 (A), J28.2 (Pin_2), Q4.3
- new net: Q3.1, R22.2, R23.1
- new net +BATT: D1.1 (K), D2.1 (K), D3.1 (K), D4.1 (K), J25.1 (Pin_1), J26.1 (Pin_1), J27.1 (Pin_1), J28.1 (Pin_1)
- new net S2: R20.1
- new net S3: R22.1
- new net S4: R24.1

Commit message: Revmoed Diodes (Built in to MOSFET)
Parts:
- removed D1, D2, D3, D4: D, Diode_SMD:D_SOD-123, symbol Device:D

Commit message: Removed extraneous Resistors
Parts:
- removed R18, R20, R22, R24: 160, Resistor_SMD:R_0603_1608Metric, symbol Device:R
- removed R19, R21, R23, R25: 100k, Resistor_SMD:R_0603_1608Metric, symbol Device:R
- added D1, D2, D3, D4: D, Diode_SMD:D_SMA, symbol Device:D
Connections:
- net +BATT: now also D1.1 (K), D2.1 (K), D3.1 (K), D4.1 (K)
- net GND: now also Q1.1, Q2.1, Q3.1, Q4.1
- net at J25.2 (Pin_2), Q1.3: now also D1.2 (A)
- net at J26.2 (Pin_2), Q2.3: now also D2.2 (A)
- net at J27.2 (Pin_2), Q3.3: now also D3.2 (A)
- net at J28.2 (Pin_2), Q4.3: now also D4.2 (A)

Commit message: Added Power Status LEDs
Connections:
- net GND: no longer Q1.1, Q2.1, Q3.1, Q4.1
- new net S1: Q1.1
- new net S2: Q2.1
- new net S3: Q3.1
- new net S4: Q4.1
Other:
- moved on the sheet: D1, D3, D4, J25, J27, J28, Q1, Q3, Q4

Commit message: read description
Other:
- moved on the sheet: D1, D2, D3, D4, J25, J26, J27, J28, Q1, Q2, Q3, Q4

Commit message: estop added
Parts:
- added J33: Conn_01x02, BM02B-GHS:JST_BM02B-GHS-TBT_LF__SN_, symbol Connector_Generic:Conn_01x02
- added JP1: SolderJumper_2_Open, Jumper:SolderJumper-2_P1.3mm_Open_TrianglePad1.0x1.5mm, symbol Jumper:SolderJumper_2_Open
Connections:
- net +BATT: now also J33.1 (Pin_1), JP1.1 (A); no longer D1.1 (K), D2.1 (K), D3.1 (K), D4.1 (K), J25.1 (Pin_1), J26.1 (Pin_1), J27.1 (Pin_1), J28.1 (Pin_1)
- new net SW_PWR: D1.1 (K), D2.1 (K), D3.1 (K), D4.1 (K), J25.1 (Pin_1), J26.1 (Pin_1), J27.1 (Pin_1), J28.1 (Pin_1), J33.2 (Pin_2), JP1.2 (B)
Other:
- note added: "PWR_ENABLE"
- moved on the sheet: D1, D2, D3, D4, J25, J26, J27, J28, Q1, Q2, Q3, Q4

Commit message: added leds🔴🟡🔵
Parts:
- renumbered D1 to D5, D2 to D6, D3 to D7, D4 to D8, J33 to J25, J25 to J26, J26 to J27, J27 to J28, J28 to J29
Changed lines of the file:
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@@
 		(dnp no)
 		(fields_autoplaced yes)
-		(property "Reference" "J25"
+		(property "Reference" "J26"
 			(at 134.62 82.5499 0)
 			(effects
@@
 			(project "Alpha_Breakout"
 				(path "/bb73515c-a1ce-4448-8899-3a433fb04c26/2e0053fd-4344-479e-8bb9-1383fd6257db"
-					(reference "J25")
+					(reference "J26")
 					(unit 1)
 				)
@@
 		(dnp no)
 		(fields_autoplaced yes)
-		(property "Reference" "D4"
+		(property "Reference" "D8"
 			(at 250.19 86.3599 90)
 			(effects
@@
 			(project "Alpha_Breakout"
 				(path "/bb73515c-a1ce-4448-8899-3a433fb04c26/2e0053fd-4344-479e-8bb9-1383fd6257db"
-					(reference "D4")
+					(reference "D8")
 					(unit 1)
 				)
@@
 		(dnp no)
 		(fields_autoplaced yes)
-		(property "Reference" "#PWR098"
+		(property "Reference" "#PWR0101"
 			(at 162.56 123.19 0)
 			(effects
@@
 			(project "Alpha_Breakout"
 				(path "/bb73515c-a1ce-4448-8899-3a433fb04c26/2e0053fd-4344-479e-8bb9-1383fd6257db"
-					(reference "#PWR098")
+					(reference "#PWR0101")
 					(unit 1)
 				)
@@
 		(dnp no)
 		(fields_autoplaced yes)
-		(property "Reference" "J33"
+		(property "Reference" "J25"
 			(at 62.23 97.7899 0)
 			(effects
@@
 			(project ""
 				(path "/bb73515c-a1ce-4448-8899-3a433fb04c26/2e0053fd-4344-479e-8bb9-1383fd6257db"
-					(reference "J33")
+					(reference "J25")
 					(unit 1)
 				)
@@
 		(dnp no)
 		(fields_autoplaced yes)
-		(property "Reference" "D2"
+		(property "Reference" "D6"
 			(at 166.37 85.0899 90)
 			(effects
@@
 			(project "Alpha_Breakout"
 				(path "/bb73515c-a1ce-4448-8899-3a433fb04c26/2e0053fd-4344-479e-8bb9-1383fd6257db"
-					(reference "D2")
+					(reference "D6")
 					(unit 1)
 				)
@@
 		(dnp no)
 		(fields_autoplaced yes)
-		(property "Reference" "J26"
+		(property "Reference" "J27"
 			(at 176.53 82.5499 0)
 			(effects
@@
 			(project "Alpha_Breakout"
 				(path "/bb73515c-a1ce-4448-8899-3a433fb04c26/2e0053fd-4344-479e-8bb9-1383fd6257db"
-					(reference "J26")
+					(reference "J27")
 					(unit 1)
 				)
@@
 		(dnp no)
 		(fields_autoplaced yes)
-		(property "Reference" "J27"
+		(property "Reference" "J28"
 			(at 218.44 83.8199 0)
 			(effects
@@
 			(project "Alpha_Breakout"
 				(path "/bb73515c-a1ce-4448-8899-3a433fb04c26/2e0053fd-4344-479e-8bb9-1383fd6257db"
-					(reference "J27")
+					(reference "J28")
 					(unit 1)
 				)
@@
 		(dnp no)
 		(fields_autoplaced yes)
-		(property "Reference" "D3"
+		(property "Reference" "D7"
 			(at 208.28 86.3599 90)
 			(effects
@@
 			(project "Alpha_Breakout"
 				(path "/bb73515c-a1ce-4448-8899-3a433fb04c26/2e0053fd-4344-479e-8bb9-1383fd6257db"
-					(reference "D3")
+					(reference "D7")
 					(unit 1)
 				)
@@
 		(dnp no)
 		(fields_autoplaced yes)
-		(property "Reference" "#PWR096"
+		(property "Reference" "#PWR0100"
 			(at 120.65 123.19 0)
 			(effects
@@
 			(project ""
 				(path "/bb73515c-a1ce-4448-8899-3a433fb04c26/2e0053fd-4344-479e-8bb9-1383fd6257db"
-					(reference "#PWR096")
+					(reference "#PWR0100")
 					(unit 1)
 				)
@@
 		(dnp no)
 		(fields_autoplaced yes)
-		(property "Reference" "D1"
+		(property "Reference" "D5"
 			(at 124.46 83.8199 90)
 			(effects
@@
 			(project ""
 				(path "/bb73515c-a1ce-4448-8899-3a433fb04c26/2e0053fd-4344-479e-8bb9-1383fd6257db"
-					(reference "D1")
+					(reference "D5")
 					(unit 1)
 				)
@@
 		(dnp no)
 		(fields_autoplaced yes)
-		(property "Reference" "#PWR0100"
+		(property "Reference" "#PWR0102"
 			(at 204.47 124.46 0)
 			(effects
@@
 			(project "Alpha_Breakout"
 				(path "/bb73515c-a1ce-4448-8899-3a433fb04c26/2e0053fd-4344-479e-8bb9-1383fd6257db"
-					(reference "#PWR0100")
+					(reference "#PWR0102")
 					(unit 1)
 				)
@@
 		(dnp no)
 		(fields_autoplaced yes)
-		(property "Reference" "#PWR0118"
+		(property "Reference" "#PWR099"
 			(at 54.61 96.52 0)
 			(effects
@@
 			(project ""
 				(path "/bb73515c-a1ce-4448-8899-3a433fb04c26/2e0053fd-4344-479e-8bb9-1383fd6257db"
-					(reference "#PWR0118")
+					(reference "#PWR099")
 					(unit 1)
 				)
@@
 		(dnp no)
 		(fields_autoplaced yes)
-		(property "Reference" "J28"
+		(property "Reference" "J29"
 			(at 260.35 83.8199 0)
 			(effects
@@
 			(project "Alpha_Breakout"
 				(path "/bb73515c-a1ce-4448-8899-3a433fb04c26/2e0053fd-4344-479e-8bb9-1383fd6257db"
-					(reference "J28")
-					(unit 1)
-				)
+					(reference "J29")
+					(unit 1)
+				)

Commit message: bunchostuff💐
Other:
- moved on the sheet: J25, JP1
Changed lines of the file:
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@@
 	(paper "A4")
 	(rectangle
-		(start 38.1 86.36)
-		(end 77.47 115.57)
+		(start 50.8 73.66)
+		(end 90.17 102.87)
 		(stroke
 			(width 0)
@@
 	(text "PWR_ENABLE"
 		(exclude_from_sim no)
-		(at 43.942 85.344 0)
+		(at 56.642 72.644 0)
 		(effects
 			(font
@@
 	)
 	(junction
-		(at 54.61 96.52)
+		(at 67.31 83.82)
 		(diameter 0)
 		(color 0 0 0 0)
@@
 	)
 	(junction
-		(at 54.61 104.14)
+		(at 67.31 91.44)
 		(diameter 0)
 		(color 0 0 0 0)
@@
 	(wire
 		(pts
-			(xy 46.99 96.52) (xy 54.61 96.52)
+			(xy 59.69 83.82) (xy 67.31 83.82)
 		)
 		(stroke
@@
 	(wire
 		(pts
-			(xy 54.61 104.14) (xy 54.61 111.76)
+			(xy 67.31 91.44) (xy 67.31 99.06)
 		)
 		(stroke
@@
 	(wire
 		(pts
-			(xy 54.61 92.71) (xy 54.61 96.52)
-		)
-		(stroke
-			(width 0)
-			(type default)
-		)
-	)
-	(wire
-		(pts
-			(xy 54.61 96.52) (xy 54.61 97.79)
+			(xy 67.31 80.01) (xy 67.31 83.82)
+		)
+		(stroke
+			(width 0)
+			(type default)
+		)
+	)
+	(wire
+		(pts
+			(xy 67.31 83.82) (xy 67.31 85.09)
 		)
 		(stroke
@@
 	(wire
 		(pts
-			(xy 54.61 100.33) (xy 54.61 104.14)
+			(xy 67.31 87.63) (xy 67.31 91.44)
 		)
 		(stroke
@@
 	(wire
 		(pts
-			(xy 46.99 104.14) (xy 54.61 104.14)
+			(xy 59.69 91.44) (xy 67.31 91.44)
 		)
 		(stroke
@@
 	(global_label "SW_PWR"
 		(shape input)
-		(at 54.61 111.76 180)
+		(at 67.31 99.06 180)
 		(fields_autoplaced yes)
 		(effects
@@
 		)
 		(property "Intersheetrefs" "${INTERSHEET_REFS}"
-			(at 44.0049 111.76 0)
+			(at 56.7049 99.06 0)
 			(effects
 				(font
@@
 	(symbol
 		(lib_id "Connector_Generic:Conn_01x02")
-		(at 59.69 97.79 0)
+		(at 72.39 85.09 0)
 		(unit 1)
 		(exclude_from_sim no)
@@
 		(fields_autoplaced yes)
 		(property "Reference" "J25"
-			(at 62.23 97.7899 0)
+			(at 74.93 85.0899 0)
 			(effects
 				(font
@@
 		)
 		(property "Value" "Conn_01x02"
-			(at 62.23 100.3299 0)
+			(at 74.93 87.6299 0)
 			(effects
 				(font
@@
 		)
 		(property "Footprint" "BM02B-GHS:JST_BM02B-GHS-TBT_LF__SN_"
-			(at 59.69 97.79 0)
+			(at 72.39 85.09 0)
 			(effects
 				(font
@@
 		)
 		(property "Datasheet" "~"
-			(at 59.69 97.79 0)
+			(at 72.39 85.09 0)
 			(effects
 				(font
@@
 		)
 		(property "Description" "Generic connector, single row, 01x02, script generated (kicad-library-utils/schlib/autogen/connector/)"
-			(at 59.69 97.79 0)
+			(at 72.39 85.09 0)
 			(effects
 				(font
@@
 	(symbol
 		(lib_id "Jumper:SolderJumper_2_Open")
-		(at 46.99 100.33 270)
+		(at 59.69 87.63 270)
 		(unit 1)
 		(exclude_from_sim no)
@@
 		(dnp no)
 		(property "Reference" "JP1"
-			(at 41.402 100.838 90)
+			(at 54.102 88.138 90)
 			(effects
 				(font
@@
 		)
 		(property "Value" "SolderJumper_2_Open"
-			(at 24.638 103.124 90)
+			(at 37.338 90.424 90)
 			(effects
 				(font
@@
 		)
 		(property "Footprint" "Jumper:SolderJumper-2_P1.3mm_Open_TrianglePad1.0x1.5mm"
-			(at 46.99 100.33 0)
+			(at 59.69 87.63 0)
 			(effects
 				(font
@@
 		)
 		(property "Datasheet" "~"
-			(at 46.99 100.33 0)
+			(at 59.69 87.63 0)
 			(effects
 				(font
@@
 		)
 		(property "Description" "Solder Jumper, 2-pole, open"
-			(at 46.99 100.33 0)
+			(at 59.69 87.63 0)
 			(effects
 				(font
@@
 	(symbol
 		(lib_id "power:+BATT")
-		(at 54.61 92.71 0)
+		(at 67.31 80.01 0)
 		(unit 1)
 		(exclude_from_sim no)
@@
 		(fields_autoplaced yes)
 		(property "Reference" "#PWR099"
-			(at 54.61 96.52 0)
+			(at 67.31 83.82 0)
 			(effects
 				(font
@@
 		)
 		(property "Value" "+BATT"
-			(at 54.61 87.63 0)
+			(at 67.31 74.93 0)
 			(effects
 				(font
@@
 		)
 		(property "Footprint" ""
-			(at 54.61 92.71 0)
+			(at 67.31 80.01 0)
 			(effects
 				(font
@@
 		)
 		(property "Datasheet" ""
-			(at 54.61 92.71 0)
+			(at 67.31 80.01 0)
 			(effects
 				(font
@@
 		)
 		(property "Description" "Power symbol creates a global label with name \"+BATT\""
-			(at 54.61 92.71 0)
-			(effects
-				(font
+			(at 67.31 80.01 0)
+			(effects
+				(font
