File: Solenoids.kicad_sch (KiCad schematic)
At the start: 14 parts, among them J25 Conn_01x02, J26 Conn_01x02, J27 Conn_01x02, J28 Conn_01x02, J29 Conn_01x02, Q1 CSD13381F4, Q2 CSD13381F4, Q3 CSD13381F4, Q4 CSD13381F4

Commit message: First Draft of BOM
Didn't select some compoentns like diodes that I don't fully understand. Also, some components have multiple variants so we must be careful.
Parts:
- J25: JLC# (none) -> C161690
- Q1, Q2, Q3, Q4: JLC# (none) -> C179868
Changed lines of the file:
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@@
+			)
+		)
+		(property "JLC#" ""
+			(at 132.08 82.55 0)
+			(effects
+				(font
+					(size 1.27 1.27)
+				)
 			)
 		)
@@
 			)
 		)
+		(property "JLC#" ""
+			(at 247.65 87.63 0)
+			(effects
+				(font
+					(size 1.27 1.27)
+				)
+			)
+		)
 		(pin "1"
 		)
@@
 			)
 		)
+		(property "JLC#" "C179868"
+			(at 160.02 99.06 0)
+			(effects
+				(font
+					(size 1.27 1.27)
+				)
+			)
+		)
 		(pin "3"
 		)
@@
 			)
 		)
+		(property "JLC#" "C161690"
+			(at 72.39 85.09 0)
+			(effects
+				(font
+					(size 1.27 1.27)
+				)
+			)
+		)
 		(pin "2"
 		)
@@
 				)
 				(hide yes)
+			)
+		)
+		(property "JLC#" ""
+			(at 59.69 87.63 0)
+			(effects
+				(font
+					(size 1.27 1.27)
+				)
 			)
 		)
@@
 			)
 		)
+		(property "JLC#" ""
+			(at 163.83 86.36 0)
+			(effects
+				(font
+					(size 1.27 1.27)
+				)
+			)
+		)
 		(pin "1"
 		)
@@
 			)
 		)
+		(property "JLC#" ""
+			(at 173.99 82.55 0)
+			(effects
+				(font
+					(size 1.27 1.27)
+				)
+			)
+		)
 		(pin "1"
 		)
@@
 			)
 		)
+		(property "JLC#" "C179868"
+			(at 118.11 99.06 0)
+			(effects
+				(font
+					(size 1.27 1.27)
+				)
+			)
+		)
 		(pin "3"
 		)
@@
 			)
 		)
+		(property "JLC#" ""
+			(at 215.9 83.82 0)
+			(effects
+				(font
+					(size 1.27 1.27)
+				)
+			)
+		)
 		(pin "1"
 		)
@@
 			)
 		)
+		(property "JLC#" ""
+			(at 205.74 87.63 0)
+			(effects
+				(font
+					(size 1.27 1.27)
+				)
+			)
+		)
 		(pin "1"
 		)
@@
 			)
 		)
+		(property "JLC#" "C179868"
+			(at 243.84 100.33 0)
+			(effects
+				(font
+					(size 1.27 1.27)
+				)
+			)
+		)
 		(pin "3"
 		)
@@
 			)
 		)
+		(property "JLC#" ""
+			(at 121.92 85.09 0)
+			(effects
+				(font
+					(size 1.27 1.27)
+				)
+			)
+		)
 		(pin "1"
 		)
@@
 			)
 		)
+		(property "JLC#" "C179868"
+			(at 201.93 100.33 0)
+			(effects
+				(font
+					(size 1.27 1.27)
+				)
+			)
+		)
 		(pin "3"
 		)
@@
 			)
 		)
+		(property "JLC#" ""
+			(at 257.81 83.82 0)
+			(effects
+				(font
+					(size 1.27 1.27)
+				)
+			)
+		)

Commit message: parts⚙️
Parts:
- D5, D6, D7, D8: JLC# (none) -> C8678
- J25: JLC# C161690 -> C161690
- J26, J27, J28, J29: JLC# (none) -> C918120
Changed lines of the file:
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@@
 			)
 		)
-		(property "JLC#" ""
+		(property "JLC#" "C918120"
 			(at 132.08 82.55 0)
 			(effects
@@
 					(size 1.27 1.27)
 				)
+				(hide yes)
 			)
 		)
@@
 			)
 		)
-		(property "JLC#" ""
+		(property "JLC#" "C8678"
 			(at 247.65 87.63 0)
 			(effects
@@
 					(size 1.27 1.27)
 				)
+				(hide yes)
 			)
 		)
@@
 					(size 1.27 1.27)
 				)
+				(hide yes)
 			)
 		)
@@
 			)
 		)
-		(property "JLC#" "C161690"
+		(property "JLC#" " C161690"
 			(at 72.39 85.09 0)
 			(effects
@@
 					(size 1.27 1.27)
 				)
+				(hide yes)
 			)
 		)
@@
 				)
 				(hide yes)
-			)
-		)
-		(property "JLC#" ""
-			(at 59.69 87.63 0)
-			(effects
-				(font
-					(size 1.27 1.27)
-				)
 			)
 		)
@@
 			)
 		)
-		(property "JLC#" ""
+		(property "JLC#" "C8678"
 			(at 163.83 86.36 0)
 			(effects
@@
 					(size 1.27 1.27)
 				)
+				(hide yes)
 			)
 		)
@@
 			)
 		)
-		(property "JLC#" ""
+		(property "JLC#" "C918120"
 			(at 173.99 82.55 0)
 			(effects
@@
 					(size 1.27 1.27)
 				)
+				(hide yes)
 			)
 		)
@@
 					(size 1.27 1.27)
 				)
+				(hide yes)
 			)
 		)
@@
 			)
 		)
-		(property "JLC#" ""
+		(property "JLC#" "C918120"
 			(at 215.9 83.82 0)
 			(effects
@@
 					(size 1.27 1.27)
 				)
+				(hide yes)
 			)
 		)
@@
 			)
 		)
-		(property "JLC#" ""
+		(property "JLC#" "C8678"
 			(at 205.74 87.63 0)
 			(effects
@@
 					(size 1.27 1.27)
 				)
+				(hide yes)
 			)
 		)
@@
 					(size 1.27 1.27)
 				)
+				(hide yes)
 			)
 		)
@@
 			)
 		)
-		(property "JLC#" ""
+		(property "JLC#" "C8678"
 			(at 121.92 85.09 0)
 			(effects
@@
 					(size 1.27 1.27)
 				)
+				(hide yes)
 			)
 		)
@@
 					(size 1.27 1.27)
 				)
+				(hide yes)
 			)
 		)
@@
 			)
 		)
-		(property "JLC#" ""
+		(property "JLC#" "C918120"
 			(at 257.81 83.82 0)
 			(effects
@@
 					(size 1.27 1.27)
 				)
-			)
-		)
+				(hide yes)
+			)
+		)

Commit message: changed noid fets🎚️
Parts:
- removed Q1, Q2, Q3, Q4: CSD13381F4, CSD13381F4:DFN100X60X35-3N, symbol CSD13381F4:CSD13381F4
- added Q1, Q2, Q3, Q4: NMOS, SI2302:SOT23, symbol Simulation_SPICE:NMOS
Connections:
- net GND: now also Q1.3 (S), Q2.3 (S), Q3.3 (S), Q4.3 (S)
- net S1: now also Q1.2 (G)
- net S2: now also Q2.2 (G)
- net S3: now also Q3.2 (G)
- net S4: now also Q4.2 (G)
- net at D5.2 (A), J26.2 (Pin_2): now also Q1.1 (D)
- net at D8.2 (A), J29.2 (Pin_2): now also Q4.1 (D)
- net at D6.2 (A), J27.2 (Pin_2): now also Q2.1 (D)
- net at D7.2 (A), J28.2 (Pin_2): now also Q3.1 (D)
