File: prog.kicad_sch (KiCad schematic)
At the start: 5 parts, among them J2 USB_C_Receptacle_USB2.0_16P, U2 CH340N

Commit message: fixed usb 🔌
Connections:
- net USB_RX: now also U2.7 (RXD); no longer TP1.1, U2.6 (TXD)
- net USB_TX: now also TP1.1, U2.6 (TXD); no longer U2.7 (RXD)
Changed lines of the file:
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@@
 	(hierarchical_label "USB_RX"
 		(shape input)
-		(at 203.2 93.98 0)
+		(at 203.2 96.52 0)
 		(effects
 			(font
@@
 	(hierarchical_label "USB_TX"
 		(shape input)
-		(at 203.2 96.52 0)
+		(at 203.2 93.98 0)
 		(effects
 			(font
