File: thermoAms.kicad_sch (KiCad schematic)
At the start: 0 parts

Commit message: Completed schematic for one IC
Parts:
- added C25, C26, C28, C29: .01uF, symbol Device:C
- added C27: .1uF, Capacitor_SMD:C_0402_1005Metric, symbol Device:C
- added J5: Conn_01x02, TerminalBlock_Phoenix:TerminalBlock_Phoenix_MKDS-1,5-2-5.08_1x02_P5.08mm_Horizontal, symbol Connector_Generic:Conn_01x02
- added R12, R13: 100, symbol Device:R
- added U9: MAX31856, Package_SO:TSSOP-14_4.4x5mm_P0.65mm, symbol Sensor_Temperature:MAX31856
Connections:
- new net: C25.2, C27.1, R12.2, U9.4 (T+)
- new net: C26.2, C27.2, R13.2, U9.3 (T-)
- new net: J5.1 (Pin_1), R13.1, U9.2 (BIAS)
- new net: J5.2 (Pin_2), R12.1
- new net +3.3V: C28.2, C29.1, U9.5 (AVDD), U9.8 (DVDD)
- new net GND: C25.1, C26.1, C28.1, C29.2, U9.1 (AGND), U9.14 (DGND)
- new net SPI1_MISO: U9.11 (SDO)
- new net SPI1_MOSI: U9.12 (SDI)
- new net SPI1_SCK: U9.10 (SCK)
- new net TC4_CS: U9.9 (~{CS})
- no-connect marks 0 -> 2

Commit message: reg🟡
Parts:
- renumbered C25 to C10, C26 to C11, C27 to C12, C28 to C13, C29 to C14, J5 to J2, R12 to R6, R13 to R7, U9 to U5
Changed lines of the file:
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@@
 		(dnp no)
 		(fields_autoplaced yes)
-		(property "Reference" "C27"
+		(property "Reference" "C12"
 			(at 210.82 119.38 90)
 			(effects
@@
 			(project "Alpha_Breakout"
 				(path "/bb73515c-a1ce-4448-8899-3a433fb04c26/7206d2b0-7b5f-4365-98b4-710ce982513e"
-					(reference "C27")
+					(reference "C12")
 					(unit 1)
 				)
@@
 		(dnp no)
 		(fields_autoplaced yes)
-		(property "Reference" "#PWR040"
+		(property "Reference" "#PWR022"
 			(at 201.93 148.59 0)
 			(effects
@@
 			(project "Alpha_Breakout"
 				(path "/bb73515c-a1ce-4448-8899-3a433fb04c26/7206d2b0-7b5f-4365-98b4-710ce982513e"
-					(reference "#PWR040")
+					(reference "#PWR022")
 					(unit 1)
 				)
@@
 		(on_board yes)
 		(dnp no)
-		(property "Reference" "C25"
+		(property "Reference" "C10"
 			(at 186.69 137.668 0)
 			(effects
@@
 			(project "Alpha_Breakout"
 				(path "/bb73515c-a1ce-4448-8899-3a433fb04c26/7206d2b0-7b5f-4365-98b4-710ce982513e"
-					(reference "C25")
+					(reference "C10")
 					(unit 1)
 				)
@@
 		(dnp no)
 		(fields_autoplaced yes)
-		(property "Reference" "#PWR041"
+		(property "Reference" "#PWR023"
 			(at 226.06 110.49 0)
 			(effects
@@
 			(project "Alpha_Breakout"
 				(path "/bb73515c-a1ce-4448-8899-3a433fb04c26/7206d2b0-7b5f-4365-98b4-710ce982513e"
-					(reference "#PWR041")
+					(reference "#PWR023")
 					(unit 1)
 				)
@@
 		(on_board yes)
 		(dnp no)
-		(property "Reference" "R13"
+		(property "Reference" "R7"
 			(at 180.594 135.89 90)
 			(effects
@@
 			(project "Alpha_Breakout"
 				(path "/bb73515c-a1ce-4448-8899-3a433fb04c26/7206d2b0-7b5f-4365-98b4-710ce982513e"
-					(reference "R13")
+					(reference "R7")
 					(unit 1)
 				)
@@
 		(on_board yes)
 		(dnp no)
-		(property "Reference" "#PWR044"
+		(property "Reference" "#PWR026"
 			(at 242.57 110.49 0)
 			(effects
@@
 			(project "Alpha_Breakout"
 				(path "/bb73515c-a1ce-4448-8899-3a433fb04c26/7206d2b0-7b5f-4365-98b4-710ce982513e"
-					(reference "#PWR044")
+					(reference "#PWR026")
 					(unit 1)
 				)
@@
 		(dnp no)
 		(fields_autoplaced yes)
-		(property "Reference" "U9"
+		(property "Reference" "U5"
 			(at 237.0933 115.57 0)
 			(effects
@@
 			(project "Alpha_Breakout"
 				(path "/bb73515c-a1ce-4448-8899-3a433fb04c26/7206d2b0-7b5f-4365-98b4-710ce982513e"
-					(reference "U9")
+					(reference "U5")
 					(unit 1)
 				)
@@
 		(dnp no)
 		(fields_autoplaced yes)
-		(property "Reference" "#PWR042"
+		(property "Reference" "#PWR024"
 			(at 234.95 105.41 0)
 			(effects
@@
 			(project "Alpha_Breakout"
 				(path "/bb73515c-a1ce-4448-8899-3a433fb04c26/7206d2b0-7b5f-4365-98b4-710ce982513e"
-					(reference "#PWR042")
+					(reference "#PWR024")
 					(unit 1)
 				)
@@
 		(dnp no)
 		(fields_autoplaced yes)
-		(property "Reference" "C29"
+		(property "Reference" "C14"
 			(at 238.76 96.52 90)
 			(effects
@@
 			(project "Alpha_Breakout"
 				(path "/bb73515c-a1ce-4448-8899-3a433fb04c26/7206d2b0-7b5f-4365-98b4-710ce982513e"
-					(reference "C29")
+					(reference "C14")
 					(unit 1)
 				)
@@
 		(dnp no)
 		(fields_autoplaced yes)
-		(property "Reference" "#PWR039"
+		(property "Reference" "#PWR021"
 			(at 194.31 148.59 0)
 			(effects
@@
 			(project "Alpha_Breakout"
 				(path "/bb73515c-a1ce-4448-8899-3a433fb04c26/7206d2b0-7b5f-4365-98b4-710ce982513e"
-					(reference "#PWR039")
+					(reference "#PWR021")
 					(unit 1)
 				)
@@
 		(dnp no)
 		(fields_autoplaced yes)
-		(property "Reference" "J5"
+		(property "Reference" "J2"
 			(at 171.45 124.46 0)
 			(effects
@@
 			(project "Alpha_Breakout"
 				(path "/bb73515c-a1ce-4448-8899-3a433fb04c26/7206d2b0-7b5f-4365-98b4-710ce982513e"
-					(reference "J5")
+					(reference "J2")
 					(unit 1)
 				)
@@
 		(dnp no)
 		(fields_autoplaced yes)
-		(property "Reference" "C28"
+		(property "Reference" "C13"
 			(at 229.87 96.52 90)
 			(effects
@@
 			(project "Alpha_Breakout"
 				(path "/bb73515c-a1ce-4448-8899-3a433fb04c26/7206d2b0-7b5f-4365-98b4-710ce982513e"
-					(reference "C28")
+					(reference "C13")
 					(unit 1)
 				)
@@
 		(dnp no)
 		(fields_autoplaced yes)
-		(property "Reference" "#PWR043"
+		(property "Reference" "#PWR025"
 			(at 234.95 161.29 0)
 			(effects
@@
 			(project "Alpha_Breakout"
 				(path "/bb73515c-a1ce-4448-8899-3a433fb04c26/7206d2b0-7b5f-4365-98b4-710ce982513e"
-					(reference "#PWR043")
+					(reference "#PWR025")
 					(unit 1)
 				)
@@
 		(dnp no)
 		(fields_autoplaced yes)
-		(property "Reference" "R12"
+		(property "Reference" "R6"
 			(at 180.34 124.46 90)
 			(effects
@@
 			(project "Alpha_Breakout"
 				(path "/bb73515c-a1ce-4448-8899-3a433fb04c26/7206d2b0-7b5f-4365-98b4-710ce982513e"
-					(reference "R12")
+					(reference "R6")
 					(unit 1)
 				)
@@
 		(dnp no)
 		(fields_autoplaced yes)
-		(property "Reference" "C26"
+		(property "Reference" "C11"
 			(at 205.74 137.1599 0)
 			(effects
@@
 			(project "Alpha_Breakout"
 				(path "/bb73515c-a1ce-4448-8899-3a433fb04c26/7206d2b0-7b5f-4365-98b4-710ce982513e"
-					(reference "C26")
-					(unit 1)
-				)
+					(reference "C11")
+					(unit 1)
+				)

Commit message: Added thermocouple footprints
8205 used in case we end up hand soldering this thing
Parts:
- added C34, C35, C37, C38, C39, C40, C42, C43, C44, C45, C47, C48: .01uF, Capacitor_SMD:C_0805_2012Metric, symbol Device:C
- added C36, C41, C46: .1uF, Capacitor_SMD:C_0805_2012Metric, symbol Device:C
- added J20, J21, J22: Conn_01x02, TerminalBlock_Phoenix:TerminalBlock_Phoenix_MKDS-1,5-2-5.08_1x02_P5.08mm_Horizontal, symbol Connector_Generic:Conn_01x02
- added R12, R13, R14, R15, R16, R17: 100, Resistor_SMD:R_0805_2012Metric, symbol Device:R
- added U10, U8, U9: MAX31856, Package_SO:TSSOP-14_4.4x5mm_P0.65mm, symbol Sensor_Temperature:MAX31856
- C10, C11, C13, C14: footprint (none) -> Capacitor_SMD:C_0805_2012Metric
- C12: footprint Capacitor_SMD:C_0402_1005Metric -> Capacitor_SMD:C_0805_2012Metric
- R6, R7: footprint (none) -> Resistor_SMD:R_0805_2012Metric
Connections:
- net +3.3V: now also C37.2, C38.1, C42.2, C43.1, C47.2, C48.1, U10.5 (AVDD), U10.8 (DVDD), U8.5 (AVDD), U8.8 (DVDD), U9.5 (AVDD), U9.8 (DVDD)
- net GND: now also C34.1, C35.1, C37.1, C38.2, C39.1, C40.1, C42.1, C43.2, C44.1, C45.1, C47.1, C48.2, U10.1 (AGND), U10.14 (DGND), U8.1 (AGND), U8.14 (DGND), U9.1 (AGND), U9.14 (DGND)
- net SPI1_MISO: now also U10.11 (SDO), U8.11 (SDO), U9.11 (SDO)
- net SPI1_MOSI: now also U10.12 (SDI), U8.12 (SDI), U9.12 (SDI)
- net SPI1_SCK: now also U10.10 (SCK), U8.10 (SCK), U9.10 (SCK)
- new net: C35.2, C36.2, R13.2, U8.3 (T-)
- new net: J20.1 (Pin_1), R13.1, U8.2 (BIAS)
- new net: J21.1 (Pin_1), R15.1, U9.2 (BIAS)
- new net: C40.2, C41.2, R15.2, U9.3 (T-)
- new net: C39.2, C41.1, R14.2, U9.4 (T+)
- new net: C44.2, C46.1, R16.2, U10.4 (T+)
- new net: J20.2 (Pin_2), R12.1
- new net: C34.2, C36.1, R12.2, U8.4 (T+)
- new net: J22.1 (Pin_1), R17.1, U10.2 (BIAS)
- new net: C45.2, C46.2, R17.2, U10.3 (T-)
- new net: J22.2 (Pin_2), R16.1
- new net: J21.2 (Pin_2), R14.1
- new net TC1_CS: U9.9 (~{CS})
- new net TC2_CS: U10.9 (~{CS})
- new net TC3_CS: U8.9 (~{CS})
- no-connect marks 2 -> 8

Commit message: thermo🌡️
Parts:
- removed C48: .01uF, Capacitor_SMD:C_0805_2012Metric, symbol Device:C
- added C1: .01uF, Capacitor_SMD:C_0402_1005Metric, symbol Device:C
- C10, C11, C13, C14, C34, C35, C37, C38, C39, C40, C42, C43, C44, C47: footprint Capacitor_SMD:C_0805_2012Metric -> Capacitor_SMD:C_0402_1005Metric
- C12, C36, C41: value .1uF -> 0.1uF; footprint Capacitor_SMD:C_0805_2012Metric -> Capacitor_SMD:C_0402_1005Metric
- C45: value .01uF -> 0.1uF; footprint Capacitor_SMD:C_0805_2012Metric -> Capacitor_SMD:C_0402_1005Metric
- C46: value .1uF -> .01uF; footprint Capacitor_SMD:C_0805_2012Metric -> Capacitor_SMD:C_0402_1005Metric
- J2, J20, J21, J22: footprint TerminalBlock_Phoenix:TerminalBlock_Phoenix_MKDS-1,5-2-5.08_1x02_P5.08mm_Horizontal -> TerminalBlock_Phoenix:TerminalBlock_Phoenix_MPT-0,5-2-2.54_1x02_P2.54mm_Horizontal
- R12, R13, R14, R15, R16, R17, R6, R7: footprint Resistor_SMD:R_0805_2012Metric -> Resistor_SMD:R_0402_1005Metric
Connections:
- net TC2_CS is gone; now on net TC1_CS: U10.9 (~{CS})
- net TC3_CS is gone; now on net TC1_CS: U8.9 (~{CS})
- net TC4_CS is gone; now on net TC1_CS: U5.9 (~{CS})
- net +3.3V: now also C46.2, C47.1; no longer C47.2
- net GND: now also C46.1, C47.2, C1.1; no longer C45.1, C47.1
- net at C41.2, R15.2, U9.3 (T-): now also C1.2; no longer C40.2
- net at R16.2, U10.4 (T+): now also C40.2, C45.1; no longer C44.2, C46.1
- net at C45.2, R17.2, U10.3 (T-): now also C44.2; no longer C46.2

Commit message: Connected solenoids, some error fixes
Connections:
- net TC1_CS: no longer U10.9 (~{CS}), U5.9 (~{CS}), U8.9 (~{CS})
- new net TC2_CS: U5.9 (~{CS})
- new net TC3_CS: U8.9 (~{CS})
- new net TC4_CS: U10.9 (~{CS})
Changed lines of the file:
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@@
 		)
 	)
-	(hierarchical_label "TC1_CS"
+	(hierarchical_label "TC4_CS"
 		(shape input)
 		(at 214.63 137.16 0)
@@
 		)
 	)
-	(hierarchical_label "TC1_CS"
+	(hierarchical_label "TC2_CS"
 		(shape input)
 		(at 215.9 58.42 0)
@@
 		)
 	)
-	(hierarchical_label "TC1_CS"
+	(hierarchical_label "TC3_CS"
 		(shape input)
 		(at 107.95 137.16 0)

Commit message: added leds🔴🟡🔵
Parts:
- renumbered C39 to C10, C34 to C11, C1 to C12, C35 to C13, C41 to C14, C36 to C15, C42 to C16, C37 to C17, C43 to C18, C38 to C19, C40 to C20, C10 to C21, C44 to C22, C11 to C23, C45 to C24, C12 to C25, C46 to C26, C13 to C27, C47 to C28, C14 to C29, J21 to J18, J20 to J19, J22 to J20, J2 to J21, R16 to R10, R17 to R11, R6 to R12, R7 to R13, R14 to R6, R15 to R7, R12 to R8, R13 to R9, U9 to U5, U8 to U6, U10 to U7, U5 to U8

Commit message: First Draft of BOM
Didn't select some compoentns like diodes that I don't fully understand. Also, some components have multiple variants so we must be careful.
Parts:
- U5, U6, U7, U8: JLC# (none) -> C2653162

Commit message: parts⚙️
Parts:
- J18, J19, J20, J21: JLC# (none) -> C918120
Changed lines of the file:
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@@
 			)
 		)
-		(property "JLC#" ""
+		(property "JLC#" "C918120"
 			(at 142.24 58.42 0)
 			(effects
@@
 					(size 1.27 1.27)
 				)
+				(hide yes)
 			)
 		)
@@
 			)
 		)
-		(property "JLC#" ""
+		(property "JLC#" "C918120"
 			(at 34.29 137.16 0)
 			(effects
@@
 					(size 1.27 1.27)
 				)
+				(hide yes)
 			)
 		)
@@
 					(size 1.27 1.27)
 				)
+				(hide yes)
 			)
 		)
@@
 					(size 1.27 1.27)
 				)
+				(hide yes)
 			)
 		)
@@
 					(size 1.27 1.27)
 				)
+				(hide yes)
 			)
 		)
@@
 			)
 		)
-		(property "JLC#" ""
+		(property "JLC#" "C918120"
 			(at 140.97 137.16 0)
 			(effects
@@
 					(size 1.27 1.27)
 				)
+				(hide yes)
 			)
 		)
@@
 					(size 1.27 1.27)
 				)
+				(hide yes)
 			)
 		)
@@
 			)
 		)
-		(property "JLC#" ""
+		(property "JLC#" "C918120"
 			(at 34.29 59.69 0)
 			(effects
@@
 					(size 1.27 1.27)
 				)
+				(hide yes)
 			)
 		)
