File: thermoAms.kicad_sch (KiCad schematic)
At the start: 36 parts, among them J18 Conn_01x02, J19 Conn_01x02, J20 Conn_01x02, J21 Conn_01x02, U5 MAX31856, U6 MAX31856, U7 MAX31856, U8 MAX31856

Commit message: Initial pass at finding Mouser part numbers
Parts:
- C10, C11, C12, C13, C16, C17, C18, C19, C20, C21, C22, C23, C26, C27, C28, C29: Mouser Part Number  (none) -> 581-0402X7R103KT2AT
- C14, C15, C24, C25: Mouser Part Number  (none) -> 581-0402YD104JAT2A
- R10, R11, R12, R13, R6, R7, R8, R9: Mouser Part Number  (none) -> 652-CR0402AJW-101GLF
- U5, U6, U7, U8: Mouser Part Number  (none) -> 700-MAX31856MUD+
