File: thermoAms.kicad_sch (KiCad schematic)
At the start: 36 parts, among them J18 Conn_01x02, J19 Conn_01x02, J20 Conn_01x02, J21 Conn_01x02, U5 MAX31856, U6 MAX31856, U7 MAX31856, U8 MAX31856

Commit message: bomupdate
Parts:
- R10, R11, R12, R13, R6, R7, R8, R9: value 100 -> 100Ω
Changed lines of the file:
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@@
 			)
 		)
-		(property "Value" "100"
+		(property "Value" "100Ω"
 			(at 43.434 142.24 90)
 			(effects
@@
 			)
 		)
-		(property "Value" "100"
+		(property "Value" "100Ω"
 			(at 150.114 142.24 90)
 			(effects
@@
 			)
 		)
-		(property "Value" "100"
+		(property "Value" "100Ω"
 			(at 43.434 64.77 90)
 			(effects
@@
 			)
 		)
-		(property "Value" "100"
+		(property "Value" "100Ω"
 			(at 43.18 130.81 90)
 			(effects
@@
 			)
 		)
-		(property "Value" "100"
+		(property "Value" "100Ω"
 			(at 151.384 63.5 90)
 			(effects
@@
 			)
 		)
-		(property "Value" "100"
+		(property "Value" "100Ω"
 			(at 149.86 130.81 90)
 			(effects
@@
 			)
 		)
-		(property "Value" "100"
+		(property "Value" "100Ω"
 			(at 151.13 52.07 90)
 			(effects
@@
 			)
 		)
-		(property "Value" "100"
+		(property "Value" "100Ω"
 			(at 43.18 53.34 90)
 			(effects
