File: ADS1231.kicad_sch (KiCad schematic)
At the start: 1 part, among them U13 ADS1231ID

Commit message: Added Load Cell IC and Circuitry, fixed wacked out symbol
Parts:
- added C49: .1uf, Capacitor_SMD:C_0402_1005Metric, symbol Device:C
- added C50, C51: 1uf, Capacitor_SMD:C_0402_1005Metric, symbol Device:C
- added J33: Conn_01x04, symbol Connector_Generic:Conn_01x04
- added R24: 10k, Resistor_SMD:R_0402_1005Metric, symbol Device:R
Connections:
- net +3.3V: now reaches U13.1 (DVDD)
- net +3.3V: now also C51.2
- net +5V: now reaches U13.10 (VREFP)
- net +5V: now also U13.13 (AVDD), C50.1, J33.4 (Pin_4), R24.1
- net GND: now reaches U13.11 (SGND), U13.2 (GND)
- net GND: now also U13.3 (CLKIN), U13.9 (VREFN), C50.2, C51.1, J33.3 (Pin_3)
- net at U13.14 (~{PDWN}): now also U13.4 (SPEED), R24.2
- net LC_SCLK: now reaches U13.15 (SCLK)
- net LC_DRDY/DOUT: now reaches U13.16 (~{DRDY}/DOUT)
- net at U13.5 (CAP): now also C49.2; no longer U13.6 (CAP)
- net at U13.7 (AINP): now also J33.2 (Pin_2)
- net at U13.8 (AINN): now also J33.1 (Pin_1)
- new net: C49.1, U13.6 (CAP)

Commit message: added leds🔴🟡🔵
Parts:
- C48: renamed from C49; value .1uf -> 0.1uF
- renumbered C50 to C49, C51 to C50, J33 to J30, R24 to R22, U13 to U12
Changed lines of the file:
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@@
 		(dnp no)
 		(fields_autoplaced yes)
-		(property "Reference" "U13"
+		(property "Reference" "U12"
 			(at 137.16 71.12 0)
 			(effects
@@
 			(project ""
 				(path "/bb73515c-a1ce-4448-8899-3a433fb04c26/735e38ae-5821-41a3-94ab-8045f709fb34"
-					(reference "U13")
+					(reference "U12")
 					(unit 1)
 				)
@@
 		(dnp no)
 		(fields_autoplaced yes)
-		(property "Reference" "#PWR0118"
+		(property "Reference" "#PWR0104"
 			(at 99.06 86.36 0)
 			(effects
@@
 			(project ""
 				(path "/bb73515c-a1ce-4448-8899-3a433fb04c26/735e38ae-5821-41a3-94ab-8045f709fb34"
-					(reference "#PWR0118")
+					(reference "#PWR0104")
 					(unit 1)
 				)
@@
 		(dnp no)
 		(fields_autoplaced yes)
-		(property "Reference" "#PWR0121"
+		(property "Reference" "#PWR0107"
 			(at 160.02 81.28 0)
 			(effects
@@
 			(project ""
 				(path "/bb73515c-a1ce-4448-8899-3a433fb04c26/735e38ae-5821-41a3-94ab-8045f709fb34"
-					(reference "#PWR0121")
+					(reference "#PWR0107")
 					(unit 1)
 				)
@@
 		(dnp no)
 		(fields_autoplaced yes)
-		(property "Reference" "R24"
+		(property "Reference" "R22"
 			(at 105.41 80.01 90)
 			(effects
@@
 			(project ""
 				(path "/bb73515c-a1ce-4448-8899-3a433fb04c26/735e38ae-5821-41a3-94ab-8045f709fb34"
-					(reference "R24")
+					(reference "R22")
 					(unit 1)
 				)
@@
 		(dnp no)
 		(fields_autoplaced yes)
-		(property "Reference" "C49"
+		(property "Reference" "C48"
 			(at 115.57 110.49 90)
 			(effects
@@
 			)
 		)
-		(property "Value" ".1uf"
+		(property "Value" "0.1uF"
 			(at 115.57 113.03 90)
 			(effects
@@
 			(project ""
 				(path "/bb73515c-a1ce-4448-8899-3a433fb04c26/735e38ae-5821-41a3-94ab-8045f709fb34"
-					(reference "C49")
+					(reference "C48")
 					(unit 1)
 				)
@@
 		(dnp no)
 		(fields_autoplaced yes)
-		(property "Reference" "C50"
+		(property "Reference" "C49"
 			(at 157.48 96.5199 0)
 			(effects
@@
 			(project "Alpha_Breakout"
 				(path "/bb73515c-a1ce-4448-8899-3a433fb04c26/735e38ae-5821-41a3-94ab-8045f709fb34"
-					(reference "C50")
+					(reference "C49")
 					(unit 1)
 				)
@@
 		(dnp no)
 		(fields_autoplaced yes)
-		(property "Reference" "#PWR0119"
+		(property "Reference" "#PWR0105"
 			(at 99.06 115.57 0)
 			(effects
@@
 			(project ""
 				(path "/bb73515c-a1ce-4448-8899-3a433fb04c26/735e38ae-5821-41a3-94ab-8045f709fb34"
-					(reference "#PWR0119")
+					(reference "#PWR0105")
 					(unit 1)
 				)
@@
 		(dnp no)
 		(fields_autoplaced yes)
-		(property "Reference" "#PWR0122"
+		(property "Reference" "#PWR0108"
 			(at 163.83 123.19 0)
 			(effects
@@
 			(project "Alpha_Breakout"
 				(path "/bb73515c-a1ce-4448-8899-3a433fb04c26/735e38ae-5821-41a3-94ab-8045f709fb34"
-					(reference "#PWR0122")
+					(reference "#PWR0108")
 					(unit 1)
 				)
@@
 		(dnp no)
 		(fields_autoplaced yes)
-		(property "Reference" "C51"
+		(property "Reference" "C50"
 			(at 167.64 96.5199 0)
 			(effects
@@
 			(project "Alpha_Breakout"
 				(path "/bb73515c-a1ce-4448-8899-3a433fb04c26/735e38ae-5821-41a3-94ab-8045f709fb34"
-					(reference "C51")
+					(reference "C50")
 					(unit 1)
 				)
@@
 		(dnp no)
 		(fields_autoplaced yes)
-		(property "Reference" "#PWR0123"
+		(property "Reference" "#PWR0106"
 			(at 160.02 78.74 0)
 			(effects
@@
 			(project ""
 				(path "/bb73515c-a1ce-4448-8899-3a433fb04c26/735e38ae-5821-41a3-94ab-8045f709fb34"
-					(reference "#PWR0123")
+					(reference "#PWR0106")
 					(unit 1)
 				)
@@
 		(dnp no)
 		(fields_autoplaced yes)
-		(property "Reference" "J33"
+		(property "Reference" "J30"
 			(at 90.17 80.01 0)
 			(effects
@@
 			(project ""
 				(path "/bb73515c-a1ce-4448-8899-3a433fb04c26/735e38ae-5821-41a3-94ab-8045f709fb34"
-					(reference "J33")
-					(unit 1)
-				)
+					(reference "J30")
+					(unit 1)
+				)

Commit message: lots🅿️
Parts:
- removed R22: 10k, Resistor_SMD:R_0402_1005Metric, symbol Device:R
Connections:
- net +3.3V: now also U12.14 (~{PDWN}), U12.4 (SPEED)
- net GND: now also J30.1 (Pin_1), U12.12 (PSW); no longer J30.3 (Pin_3)
- net at U12.8 (AINN): now also J30.3 (Pin_3); no longer J30.1 (Pin_1)
Other:
- moved on the sheet: C48, C49, C50, J30, U12

Commit message: done ✅
Parts:
- J30: footprint (none) -> SM04B-GHS:JST_SM04B-GHS-TB_LF__SN_-
Changed lines of the file:
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@@
 			)
 		)
-		(property "Footprint" ""
+		(property "Footprint" "SM04B-GHS:JST_SM04B-GHS-TB_LF__SN_-"
 			(at 100.33 91.44 0)
 			(effects

Commit message: First Draft of BOM
Didn't select some compoentns like diodes that I don't fully understand. Also, some components have multiple variants so we must be careful.
Parts:
- J30: JLC# (none) -> C189895
- U12: JLC# (none) -> C486034
Changed lines of the file:
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@@
+			)
+		)
+		(property "JLC#" "C486034"
+			(at 147.32 99.06 0)
+			(effects
+				(font
+					(size 1.27 1.27)
+				)
 			)
 		)
@@
 				)
 				(hide yes)
+			)
+		)
+		(property "JLC#" ""
+			(at 125.73 118.11 0)
+			(effects
+				(font
+					(size 1.27 1.27)
+				)
 			)
 		)
@@
 			)
 		)
+		(property "JLC#" ""
+			(at 163.83 97.79 0)
+			(effects
+				(font
+					(size 1.27 1.27)
+				)
+			)
+		)
 		(pin "2"
 		)
@@
 			)
 		)
+		(property "JLC#" ""
+			(at 173.99 97.79 0)
+			(effects
+				(font
+					(size 1.27 1.27)
+				)
+			)
+		)
 		(pin "2"
 		)
@@
 			)
 		)
+		(property "JLC#" "C189895"
+			(at 100.33 91.44 0)
+			(effects
+				(font
+					(size 1.27 1.27)
+				)
+			)
+		)

Commit message: parts⚙️
Parts:
- U12: JLC# C486034 -> C486034
Changed lines of the file:
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@@
 			)
 		)
-		(property "JLC#" "C486034"
+		(property "JLC#" "C486034 "
 			(at 147.32 99.06 0)
 			(effects
@@
 					(size 1.27 1.27)
 				)
+				(hide yes)
 			)
 		)
@@
 					(size 1.27 1.27)
 				)
-			)
-		)
+				(hide yes)
+			)
+		)

Commit message: Initial pass at finding Mouser part numbers
Parts:
- C48: Mouser Part Number  (none) -> 581-0402YD104JAT2A
- C49, C50: Mouser Part Number  (none) -> 581-04023D105KAT2A
- U12: Mouser Part Number  (none) -> 595-ADS1231ID
Changed lines of the file:
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@@
+			)
+		)
+		(property "Mouser Part Number " "595-ADS1231ID "
+			(at 147.32 99.06 0)
+			(effects
+				(font
+					(size 1.27 1.27)
+				)
 			)
 		)
@@
 		)
 		(property "JLC#" ""
+			(at 125.73 118.11 0)
+			(effects
+				(font
+					(size 1.27 1.27)
+				)
+			)
+		)
+		(property "Mouser Part Number " "581-0402YD104JAT2A "
 			(at 125.73 118.11 0)
 			(effects
@@
 			)
 		)
+		(property "Mouser Part Number " "581-04023D105KAT2A "
+			(at 163.83 97.79 0)
+			(effects
+				(font
+					(size 1.27 1.27)
+				)
+			)
+		)
 		(pin "2"
 		)
@@
 			)
 		)
+		(property "Mouser Part Number " "581-04023D105KAT2A "
+			(at 173.99 97.79 0)
+			(effects
+				(font
+					(size 1.27 1.27)
+				)
+			)
+		)
 		(pin "2"
 		)
@@
 			)
 		)
+		(property "Mouser Part Number " ""
+			(at 100.33 91.44 0)
+			(effects
+				(font
+					(size 1.27 1.27)
+				)
+			)
+		)
