File: Hardware_Safe.kicad_sch (KiCad schematic)
At the start: 6 parts, among them J29 Conn_01x02, J31 Conn_01x02, J32 Conn_01x02

Commit message: added leds🔴🟡🔵
Parts:
- renumbered J29 to J31, J31 to J32, J32 to J33, R22 to R23, R23 to R24, R27 to R25
Changed lines of the file:
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@@
 		(dnp no)
 		(fields_autoplaced yes)
-		(property "Reference" "#PWR0111"
+		(property "Reference" "#PWR0109"
 			(at 92.71 88.9 0)
 			(effects
@@
 			(project ""
 				(path "/bb73515c-a1ce-4448-8899-3a433fb04c26/1d3635ca-ff21-408a-be61-931c18b65b0c"
-					(reference "#PWR0111")
+					(reference "#PWR0109")
 					(unit 1)
 				)
@@
 		(dnp no)
 		(fields_autoplaced yes)
-		(property "Reference" "R23"
+		(property "Reference" "R24"
 			(at 123.19 97.7899 0)
 			(effects
@@
 			(project "Alpha_Breakout"
 				(path "/bb73515c-a1ce-4448-8899-3a433fb04c26/1d3635ca-ff21-408a-be61-931c18b65b0c"
-					(reference "R23")
+					(reference "R24")
 					(unit 1)
 				)
@@
 		(dnp no)
 		(fields_autoplaced yes)
-		(property "Reference" "R27"
+		(property "Reference" "R25"
 			(at 182.88 100.3299 0)
 			(effects
@@
 			(project "Alpha_Breakout"
 				(path "/bb73515c-a1ce-4448-8899-3a433fb04c26/1d3635ca-ff21-408a-be61-931c18b65b0c"
-					(reference "R27")
+					(reference "R25")
 					(unit 1)
 				)
@@
 		(dnp no)
 		(fields_autoplaced yes)
-		(property "Reference" "R22"
+		(property "Reference" "R23"
 			(at 95.25 97.7899 0)
 			(effects
@@
 			(project ""
 				(path "/bb73515c-a1ce-4448-8899-3a433fb04c26/1d3635ca-ff21-408a-be61-931c18b65b0c"
-					(reference "R22")
+					(reference "R23")
 					(unit 1)
 				)
@@
 		(dnp no)
 		(fields_autoplaced yes)
-		(property "Reference" "#PWR0112"
+		(property "Reference" "#PWR0111"
 			(at 120.65 88.9 0)
 			(effects
@@
 			(project "Alpha_Breakout"
 				(path "/bb73515c-a1ce-4448-8899-3a433fb04c26/1d3635ca-ff21-408a-be61-931c18b65b0c"
-					(reference "#PWR0112")
+					(reference "#PWR0111")
 					(unit 1)
 				)
@@
 		(dnp no)
 		(fields_autoplaced yes)
-		(property "Reference" "#PWR0113"
+		(property "Reference" "#PWR0112"
 			(at 120.65 110.49 0)
 			(effects
@@
 			(project "Alpha_Breakout"
 				(path "/bb73515c-a1ce-4448-8899-3a433fb04c26/1d3635ca-ff21-408a-be61-931c18b65b0c"
-					(reference "#PWR0113")
+					(reference "#PWR0112")
 					(unit 1)
 				)
@@
 		(dnp no)
 		(fields_autoplaced yes)
-		(property "Reference" "#PWR0114"
+		(property "Reference" "#PWR0113"
 			(at 180.34 91.44 0)
 			(effects
@@
 			(project "Alpha_Breakout"
 				(path "/bb73515c-a1ce-4448-8899-3a433fb04c26/1d3635ca-ff21-408a-be61-931c18b65b0c"
-					(reference "#PWR0114")
+					(reference "#PWR0113")
 					(unit 1)
 				)
@@
 		(dnp no)
 		(fields_autoplaced yes)
-		(property "Reference" "#PWR0115"
+		(property "Reference" "#PWR0114"
 			(at 180.34 113.03 0)
 			(effects
@@
 			(project "Alpha_Breakout"
 				(path "/bb73515c-a1ce-4448-8899-3a433fb04c26/1d3635ca-ff21-408a-be61-931c18b65b0c"
-					(reference "#PWR0115")
+					(reference "#PWR0114")
 					(unit 1)
 				)
@@
 		(dnp no)
 		(fields_autoplaced yes)
-		(property "Reference" "J31"
+		(property "Reference" "J32"
 			(at 129.54 91.4399 0)
 			(effects
@@
 			(project "Alpha_Breakout"
 				(path "/bb73515c-a1ce-4448-8899-3a433fb04c26/1d3635ca-ff21-408a-be61-931c18b65b0c"
-					(reference "J31")
+					(reference "J32")
 					(unit 1)
 				)
@@
 		(dnp no)
 		(fields_autoplaced yes)
-		(property "Reference" "J32"
+		(property "Reference" "J33"
 			(at 189.23 93.9799 0)
 			(effects
@@
 			(project "Alpha_Breakout"
 				(path "/bb73515c-a1ce-4448-8899-3a433fb04c26/1d3635ca-ff21-408a-be61-931c18b65b0c"
-					(reference "J32")
+					(reference "J33")
 					(unit 1)
 				)
@@
 		(dnp no)
 		(fields_autoplaced yes)
-		(property "Reference" "J29"
+		(property "Reference" "J31"
 			(at 101.6 91.4399 0)
 			(effects
@@
 			(project ""
 				(path "/bb73515c-a1ce-4448-8899-3a433fb04c26/1d3635ca-ff21-408a-be61-931c18b65b0c"
-					(reference "J29")
-					(unit 1)
-				)
+					(reference "J31")
+					(unit 1)
+				)

Commit message: bunchostuff💐
Parts:
- removed J32: Conn_01x02, BM02B-GHS:JST_BM02B-GHS-TBT_LF__SN_, symbol Connector_Generic:Conn_01x02
- removed R24: 20k, Resistor_SMD:R_0402_1005Metric, symbol Device:R
Connections:
- net BW1: now reaches J33.2 (Pin_2), R25.1
- net K1: now reaches J31.2 (Pin_2), R23.1
Other:
- note added: "E-STOP"
- note removed: "Keys"
- moved on the sheet: J31, R23

Commit message: done ✅
Changed lines of the file:
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@@
 	(text "Burn Wire"
 		(exclude_from_sim no)
-		(at 167.386 72.39 0)
+		(at 173.228 73.66 0)
 		(effects
 			(font

Commit message: First Draft of BOM
Didn't select some compoentns like diodes that I don't fully understand. Also, some components have multiple variants so we must be careful.
Parts:
- J31, J33: JLC# (none) -> C161690
Changed lines of the file:
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@@
+			)
+		)
+		(property "JLC#" ""
+			(at 180.34 101.6 0)
+			(effects
+				(font
+					(size 1.27 1.27)
+				)
 			)
 		)
@@
 			)
 		)
+		(property "JLC#" ""
+			(at 129.54 99.06 0)
+			(effects
+				(font
+					(size 1.27 1.27)
+				)
+			)
+		)
 		(pin "1"
 		)
@@
 			)
 		)
+		(property "JLC#" "C161690"
+			(at 186.69 93.98 0)
+			(effects
+				(font
+					(size 1.27 1.27)
+				)
+			)
+		)
 		(pin "2"
 		)
@@
 			)
 		)
+		(property "JLC#" "C161690"
+			(at 135.89 91.44 0)
+			(effects
+				(font
+					(size 1.27 1.27)
+				)
+			)
+		)

Commit message: parts⚙️
Changed lines of the file:
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@@
 					(size 1.27 1.27)
 				)
+				(hide yes)
 			)
 		)
@@
 					(size 1.27 1.27)
 				)
+				(hide yes)
 			)
 		)

Commit message: Initial pass at finding Mouser part numbers
Parts:
- R23, R25: Mouser Part Number  (none) -> 71-RCA040220K0JNED
Changed lines of the file:
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@@
+			)
+		)
+		(property "Mouser Part Number " "71-RCA040220K0JNED "
+			(at 180.34 101.6 0)
+			(effects
+				(font
+					(size 1.27 1.27)
+				)
 			)
 		)
@@
 			)
 		)
+		(property "Mouser Part Number " "71-RCA040220K0JNED "
+			(at 129.54 99.06 0)
+			(effects
+				(font
+					(size 1.27 1.27)
+				)
+			)
+		)
 		(pin "1"
 		)
@@
 			)
 		)
+		(property "Mouser Part Number " ""
+			(at 186.69 93.98 0)
+			(effects
+				(font
+					(size 1.27 1.27)
+				)
+			)
+		)
 		(pin "2"
 		)
@@
 			)
 		)
+		(property "Mouser Part Number " ""
+			(at 135.89 91.44 0)
+			(effects
+				(font
+					(size 1.27 1.27)
+				)
+			)
+		)
