File: Pyro.kicad_sch (KiCad schematic)
At the start: 8 parts, among them J34 Conn_01x02, J36 Conn_01x02, Q5 SSM3J328R, Q6 L2N7002SLLT1G

Commit message: Initial pass at finding Mouser part numbers
Parts:
- Q5: Mouser Part Number  (none) -> 757-SSM3J328RLF
- R26: Mouser Part Number  (none) -> 652-ZV20K0603300NIRH
- R27: Mouser Part Number  (none) -> 810-NTCG164LH104H
Changed lines of the file:
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@@
+			)
+		)
+		(property "Mouser Part Number " ""
+			(at 72.39 83.82 0)
+			(effects
+				(font
+					(size 1.27 1.27)
+				)
 			)
 		)
@@
 			)
 		)
+		(property "Mouser Part Number " ""
+			(at 132.08 115.57 0)
+			(effects
+				(font
+					(size 1.27 1.27)
+				)
+			)
+		)
 		(pin "2"
 		)
@@
 			)
 		)
+		(property "Mouser Part Number " "652-ZV20K0603300NIRH "
+			(at 137.16 83.82 0)
+			(effects
+				(font
+					(size 1.27 1.27)
+				)
+			)
+		)
 		(pin "2"
 		)
@@
 			)
 		)
+		(property "Mouser Part Number " ""
+			(at 142.24 101.6 0)
+			(effects
+				(font
+					(size 1.27 1.27)
+				)
+			)
+		)
 		(pin "2"
 		)
@@
 		)
 		(property "JLC#" ""
+			(at 137.16 91.44 0)
+			(effects
+				(font
+					(size 1.27 1.27)
+				)
+			)
+		)
+		(property "Mouser Part Number " ""
 			(at 137.16 91.44 0)
 			(effects
@@
 			)
 		)
+		(property "Mouser Part Number " "810-NTCG164LH104H "
+			(at 144.78 91.44 0)
+			(effects
+				(font
+					(size 1.27 1.27)
+				)
+			)
+		)
 		(pin "2"
 		)
@@
 			)
 		)
+		(property "Mouser Part Number " "757-SSM3J328RLF "
+			(at 129.54 95.25 0)
+			(effects
+				(font
+					(size 1.27 1.27)
+				)
+			)
+		)
 		(pin "1"
 		)
@@
 			)
 		)
+		(property "Mouser Part Number " ""
+			(at 85.09 81.28 0)
+			(effects
+				(font
+					(size 1.27 1.27)
+				)
+			)
+		)
