File: Pyro.kicad_sch (KiCad schematic)
At the start: 6 parts, among them J30 Conn_01x02, Q5 SSM3J328R, Q6 L2N7002SLLT1G

Commit message: added leds🔴🟡🔵
Parts:
- renumbered J30 to J34, R25 to R26, R26 to R27
Changed lines of the file:
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@@
 		(dnp no)
 		(fields_autoplaced yes)
-		(property "Reference" "J30"
+		(property "Reference" "J34"
 			(at 134.62 114.2999 90)
 			(effects
@@
 			(project "Alpha_Breakout"
 				(path "/bb73515c-a1ce-4448-8899-3a433fb04c26/972d75bc-2192-4dfc-9be4-cbf40905f0e9"
-					(reference "J30")
+					(reference "J34")
 					(unit 1)
 				)
@@
 		(dnp no)
 		(fields_autoplaced yes)
-		(property "Reference" "R25"
+		(property "Reference" "R26"
 			(at 139.7 82.5499 0)
 			(effects
@@
 			(project "Alpha_Breakout"
 				(path "/bb73515c-a1ce-4448-8899-3a433fb04c26/972d75bc-2192-4dfc-9be4-cbf40905f0e9"
-					(reference "R25")
+					(reference "R26")
 					(unit 1)
 				)
@@
 		(dnp no)
 		(fields_autoplaced yes)
-		(property "Reference" "#PWR0116"
+		(property "Reference" "#PWR0115"
 			(at 132.08 82.55 0)
 			(effects
@@
 			(project "Alpha_Breakout"
 				(path "/bb73515c-a1ce-4448-8899-3a433fb04c26/972d75bc-2192-4dfc-9be4-cbf40905f0e9"
-					(reference "#PWR0116")
+					(reference "#PWR0115")
 					(unit 1)
 				)
@@
 		(dnp no)
 		(fields_autoplaced yes)
-		(property "Reference" "R26"
+		(property "Reference" "R27"
 			(at 147.32 90.1699 0)
 			(effects
@@
 			(project "Alpha_Breakout"
 				(path "/bb73515c-a1ce-4448-8899-3a433fb04c26/972d75bc-2192-4dfc-9be4-cbf40905f0e9"
-					(reference "R26")
+					(reference "R27")
 					(unit 1)
 				)
@@
 		(dnp no)
 		(fields_autoplaced yes)
-		(property "Reference" "#PWR0117"
+		(property "Reference" "#PWR0116"
 			(at 149.86 120.65 0)
 			(effects
@@
 			(project "Alpha_Breakout"
 				(path "/bb73515c-a1ce-4448-8899-3a433fb04c26/972d75bc-2192-4dfc-9be4-cbf40905f0e9"
-					(reference "#PWR0117")
-					(unit 1)
-				)
+					(reference "#PWR0116")
+					(unit 1)
+				)

Commit message: bunchostuff💐
Parts:
- added J36: Conn_01x02, BM02B-GHS:JST_BM02B-GHS-TBT_LF__SN_, symbol Connector_Generic:Conn_01x02
- added JP2: SolderJumper_2_Open, Jumper:SolderJumper-2_P1.3mm_Open_TrianglePad1.0x1.5mm, symbol Jumper:SolderJumper_2_Open
- J34: footprint TerminalBlock_Phoenix:TerminalBlock_Phoenix_MKDS-1,5-2-5.08_1x02_P5.08mm_Horizontal -> SM02B-GHS:CONN_SM02B-GHS_JST
Connections:
- net +BATT: now also J36.1 (Pin_1), JP2.1 (A); no longer Q5.3 (S), R26.1
- new net PYRO_PWR: J36.2 (Pin_2), JP2.2 (B), Q5.3 (S), R26.1
Other:
- note added: "PYRO KEY"

Commit message: done ✅
Parts:
- J34: footprint SM02B-GHS:CONN_SM02B-GHS_JST -> Connector_PinHeader_2.54mm:PinHeader_1x02_P2.54mm_Vertical
- J36: footprint BM02B-GHS:JST_BM02B-GHS-TBT_LF__SN_ -> Connector_JST:JST_XH_B2B-XH-A_1x02_P2.50mm_Vertical
Changed lines of the file:
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@@
 			)
 		)
-		(property "Footprint" "SM02B-GHS:CONN_SM02B-GHS_JST"
+		(property "Footprint" "Connector_PinHeader_2.54mm:PinHeader_1x02_P2.54mm_Vertical"
 			(at 132.08 115.57 0)
 			(effects
@@
 			)
 		)
-		(property "Footprint" "BM02B-GHS:JST_BM02B-GHS-TBT_LF__SN_"
+		(property "Footprint" "Connector_JST:JST_XH_B2B-XH-A_1x02_P2.50mm_Vertical"
 			(at 85.09 81.28 0)
 			(effects

Commit message: First Draft of BOM
Didn't select some compoentns like diodes that I don't fully understand. Also, some components have multiple variants so we must be careful.
Parts:
- J34: JLC# (none) -> C5116481
- J36: JLC# (none) -> C158012
- Q5: JLC# (none) -> C396016
- Q6: JLC# (none) -> C22446827
Changed lines of the file:
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@@
+			)
+		)
+		(property "JLC#" ""
+			(at 72.39 83.82 0)
+			(effects
+				(font
+					(size 1.27 1.27)
+				)
 			)
 		)
@@
 			)
 		)
+		(property "JLC#" "C5116481"
+			(at 132.08 115.57 0)
+			(effects
+				(font
+					(size 1.27 1.27)
+				)
+			)
+		)
 		(pin "2"
 		)
@@
 			)
 		)
+		(property "JLC#" ""
+			(at 137.16 83.82 0)
+			(effects
+				(font
+					(size 1.27 1.27)
+				)
+			)
+		)
 		(pin "2"
 		)
@@
 			)
 		)
+		(property "JLC#" "C22446827"
+			(at 142.24 101.6 0)
+			(effects
+				(font
+					(size 1.27 1.27)
+				)
+			)
+		)
 		(pin "2"
 		)
@@
 				)
 				(hide yes)
+			)
+		)
+		(property "JLC#" ""
+			(at 137.16 91.44 0)
+			(effects
+				(font
+					(size 1.27 1.27)
+				)
 			)
 		)
@@
 			)
 		)
+		(property "JLC#" ""
+			(at 144.78 91.44 0)
+			(effects
+				(font
+					(size 1.27 1.27)
+				)
+			)
+		)
 		(pin "2"
 		)
@@
 			)
 		)
+		(property "JLC#" "C396016"
+			(at 129.54 95.25 0)
+			(effects
+				(font
+					(size 1.27 1.27)
+				)
+			)
+		)
 		(pin "1"
 		)
@@
 			)
 		)
+		(property "JLC#" "C158012"
+			(at 85.09 81.28 0)
+			(effects
+				(font
+					(size 1.27 1.27)
+				)
+			)
+		)

Commit message: parts⚙️
Parts:
- J34: JLC# C5116481 -> (none)
Changed lines of the file:
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@@
-			)
-		)
-		(property "JLC#" "C5116481"
-			(at 132.08 115.57 0)
-			(effects
-				(font
-					(size 1.27 1.27)
-				)
 			)
 		)
@@
 					(size 1.27 1.27)
 				)
+				(hide yes)
 			)
 		)
@@
 					(size 1.27 1.27)
 				)
+				(hide yes)
 			)
 		)
@@
 					(size 1.27 1.27)
 				)
-			)
-		)
+				(hide yes)
+			)
+		)

Commit message: done
Parts:
- R26: value 200k -> 100k
- R27: value 100k -> 200k
Changed lines of the file:
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@@
 			)
 		)
-		(property "Value" "200k"
+		(property "Value" "100k"
 			(at 139.7 85.0899 0)
 			(effects
@@
 			)
 		)
-		(property "Value" "100k"
+		(property "Value" "200k"
 			(at 147.32 92.7099 0)
 			(effects
