File: RS-485.kicad_sch (KiCad schematic)
At the start: 2 parts, among them J23 Conn_01x02, U11 SP3485EN

Commit message: First Draft of BOM
Didn't select some compoentns like diodes that I don't fully understand. Also, some components have multiple variants so we must be careful.
Parts:
- J23: JLC# (none) -> C189893
- U11: JLC# (none) -> C8963
Changed lines of the file:
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@@
+			)
+		)
+		(property "JLC#" "C189893"
+			(at 160.02 96.52 0)
+			(effects
+				(font
+					(size 1.27 1.27)
+				)
 			)
 		)
@@
 			)
 		)
+		(property "JLC#" "C8963"
+			(at 138.43 102.87 0)
+			(effects
+				(font
+					(size 1.27 1.27)
+				)
+			)
+		)

Commit message: parts⚙️
Changed lines of the file:
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@@
 					(size 1.27 1.27)
 				)
+				(hide yes)
 			)
 		)

Commit message: Initial pass at finding Mouser part numbers
Parts:
- U11: Mouser Part Number  (none) -> 701-SP3485EN-L/TR
Changed lines of the file:
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@@
+			)
+		)
+		(property "Mouser Part Number " ""
+			(at 160.02 96.52 0)
+			(effects
+				(font
+					(size 1.27 1.27)
+				)
 			)
 		)
@@
 			)
 		)
+		(property "Mouser Part Number " "701-SP3485EN-L/TR "
+			(at 138.43 102.87 0)
+			(effects
+				(font
+					(size 1.27 1.27)
+				)
+			)
+		)
